File: boardlock/power.kicad_sch (KiCad schematic)
At the start: 0 parts

Commit message: Added power library and fixed labels
Parts:
- added U2: BQ24075RGT, Package_DFN_QFN:VQFN-16-1EP_3x3mm_P0.5mm_EP1.6x1.6mm, symbol Battery_Management:BQ24075RGT
- added U7: BQ27441DRZR-G1A, Package_SON:Texas_S-PDSO-N12, symbol Battery_Management:BQ27441DRZR-G1A
- added U8: TPS630701RNMR, TPS630701RNMR:TPS630701RNMR, symbol TPS630701RNMR:TPS630701RNMR
Connections:
- new net: U2.10 (OUT), U2.11 (OUT)
- new net: U2.17 (VSS), U2.8 (VSS)
- new net: U2.2 (BAT), U2.3 (BAT)
Changed lines of the file:
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@@
 (kicad_sch (version 20230121) (generator eeschema)
   (paper "A4")
+  (symbol (lib_id "Battery_Management:BQ27441DRZR-G1A") (at 166.37 69.85 0) (unit 1)
+    (in_bom yes) (on_board yes) (dnp no) (fields_autoplaced)
+    (property "Reference" "U7" (at 166.37 52.07 0)
+      (effects (font (size 1.27 1.27)))
+    )
+    (property "Value" "BQ27441DRZR-G1A" (at 166.37 54.61 0)
+      (effects (font (size 1.27 1.27)))
+    )
+    (property "Footprint" "Package_SON:Texas_S-PDSO-N12" (at 172.72 83.82 0)
+      (effects (font (size 1.27 1.27)) (justify left) hide)
+    )
+    (property "Datasheet" "http://www.ti.com/lit/ds/symlink/bq27441-g1.pdf" (at 171.45 64.77 0)
+      (effects (font (size 1.27 1.27)) hide)
+    )
+    (pin "1")
+    (pin "10")
+    (pin "11")
+    (pin "12")
+    (pin "13")
+    (pin "2")
+    (pin "3")
+    (pin "4")
+    (pin "5")
+    (pin "6")
+    (pin "7")
+    (pin "8")
+    (pin "9")
+    (instances
+      (project "boardlock"
+        (path "/e1fc29ce-837e-4062-84d8-c7e423f9eab9/5801071c-337d-449a-92e5-5afeb5febc0d"
+          (reference "U7") (unit 1)
+        )
+      )
+    )
+  )
+  (symbol (lib_id "Battery_Management:BQ24075RGT") (at 64.77 68.58 0) (unit 1)
+    (in_bom yes) (on_board yes) (dnp no) (fields_autoplaced)
+    (property "Reference" "U2" (at 66.9641 50.8 0)
+      (effects (font (size 1.27 1.27)) (justify left))
+    )
+    (property "Value" "BQ24075RGT" (at 66.9641 53.34 0)
+      (effects (font (size 1.27 1.27)) (justify left))
+    )
+    (property "Footprint" "Package_DFN_QFN:VQFN-16-1EP_3x3mm_P0.5mm_EP1.6x1.6mm" (at 72.39 82.55 0)
+      (effects (font (size 1.27 1.27)) (justify left) hide)
+    )
+    (property "Datasheet" "http://www.ti.com/lit/ds/symlink/bq24075.pdf" (at 72.39 63.5 0)
+      (effects (font (size 1.27 1.27)) hide)
+    )
+    (pin "1")
+    (pin "10")
+    (pin "11")
+    (pin "12")
+    (pin "13")
+    (pin "14")
+    (pin "15")
+    (pin "16")
+    (pin "17")
+    (pin "2")
+    (pin "3")
+    (pin "4")
+    (pin "5")
+    (pin "6")
+    (pin "7")
+    (pin "8")
+    (pin "9")
+    (instances
+      (project "boardlock"
+        (path "/e1fc29ce-837e-4062-84d8-c7e423f9eab9/5801071c-337d-449a-92e5-5afeb5febc0d"
+          (reference "U2") (unit 1)
+        )
+      )
+    )
+  )
+  (symbol (lib_id "TPS630701RNMR:TPS630701RNMR") (at 111.76 134.62 0) (unit 1)
+    (in_bom yes) (on_board yes) (dnp no) (fields_autoplaced)
+    (property "Reference" "U8" (at 111.76 104.14 0)
+      (effects (font (size 1.524 1.524)))
+    )
+    (property "Value" "TPS630701RNMR" (at 111.76 106.68 0)
+      (effects (font (size 1.524 1.524)))
+    )
+    (property "Footprint" "TPS630701RNMR:TPS630701RNMR" (at 111.76 134.62 0)
+      (effects (font (size 1.27 1.27) italic) hide)
+    )
+    (property "Datasheet" "TPS630701RNMR" (at 111.76 134.62 0)
+      (effects (font (size 1.27 1.27) italic) hide)
+    )
+    (pin "1")
+    (pin "10")
+    (pin "11")
+    (pin "12")
+    (pin "13")
+    (pin "14")
+    (pin "15")
+    (pin "2")
+    (pin "3")
+    (pin "4")
+    (pin "5")
+    (pin "6")
+    (pin "7")
+    (pin "8")
+    (pin "9")
+    (instances
+      (project "boardlock"
+        (path "/e1fc29ce-837e-4062-84d8-c7e423f9eab9/5801071c-337d-449a-92e5-5afeb5febc0d"
+          (reference "U8") (unit 1)
+        )
+      )
+    )
+  )
 )
