File: boardlock/power.kicad_sch (KiCad schematic)
At the start: 24 parts, among them U6 TPS630701RNMR

Commit message: not sure what I changed
Other:
- note added: "Monitors battery voltage for buck-boost converter. Voltage divider calculation done at V_BATT = 3V. Buck-boost converter EN shuts off at 0.7V. V_BATT_BUCK_BOOST_EN = 0.683 @ VBATT = 3V V_BATT_BUCK_BOOST_EN = 0.7 @ VBATT = 3.075V"
- note removed: "Monitors battery voltage for buck-boost converter. Voltage divider calculation done at V_BATT = 3V. Buck-boost converter EN shuts off at 0.7V. V_BATT_BUCK_BOOST_EN = 0.683 @ VBATT = 3V"
- moved on the sheet: R?
Changed lines of the file:
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@@
   (junction (at 45.72 142.24) (diameter 0) (color 0 0 0 0)
   )
-  (junction (at 35.56 62.23) (diameter 0) (color 0 0 0 0)
+  (junction (at 33.02 64.77) (diameter 0) (color 0 0 0 0)
   )
   (junction (at 232.41 68.58) (diameter 0) (color 0 0 0 0)
@@
   (junction (at 82.55 142.24) (diameter 0) (color 0 0 0 0)
   )
-  (junction (at 35.56 50.8) (diameter 0) (color 0 0 0 0)
+  (junction (at 33.02 53.34) (diameter 0) (color 0 0 0 0)
   )
   (junction (at 102.87 78.74) (diameter 0) (color 0 0 0 0)
@@
   (junction (at 204.47 81.28) (diameter 0) (color 0 0 0 0)
   )
-  (junction (at 46.99 50.8) (diameter 0) (color 0 0 0 0)
+  (junction (at 44.45 53.34) (diameter 0) (color 0 0 0 0)
   )
   (wire (pts (xy 185.42 91.44) (xy 190.5 91.44))
@@
     (stroke (width 0) (type default))
   )
-  (wire (pts (xy 46.99 50.8) (xy 46.99 53.34))
-    (stroke (width 0) (type default))
-  )
-  (wire (pts (xy 35.56 62.23) (xy 46.99 62.23))
+  (wire (pts (xy 44.45 53.34) (xy 44.45 55.88))
+    (stroke (width 0) (type default))
+  )
+  (wire (pts (xy 33.02 64.77) (xy 44.45 64.77))
     (stroke (width 0) (type default))
   )
@@
     (stroke (width 0) (type default))
   )
-  (wire (pts (xy 35.56 48.26) (xy 35.56 50.8))
+  (wire (pts (xy 33.02 50.8) (xy 33.02 53.34))
     (stroke (width 0) (type default))
   )
@@
     (stroke (width 0) (type default))
   )
-  (wire (pts (xy 46.99 50.8) (xy 50.8 50.8))
+  (wire (pts (xy 44.45 53.34) (xy 48.26 53.34))
     (stroke (width 0) (type default))
   )
@@
     (stroke (width 0) (type default))
   )
-  (wire (pts (xy 46.99 60.96) (xy 46.99 62.23))
+  (wire (pts (xy 44.45 63.5) (xy 44.45 64.77))
     (stroke (width 0) (type default))
   )
@@
     (stroke (width 0) (type default))
   )
-  (wire (pts (xy 35.56 50.8) (xy 35.56 53.34))
+  (wire (pts (xy 33.02 53.34) (xy 33.02 55.88))
     (stroke (width 0) (type default))
   )
@@
     (stroke (width 0) (type default))
   )
-  (wire (pts (xy 35.56 60.96) (xy 35.56 62.23))
+  (wire (pts (xy 33.02 63.5) (xy 33.02 64.77))
     (stroke (width 0) (type default))
   )
@@
     (stroke (width 0) (type default))
   )
-  (wire (pts (xy 35.56 38.1) (xy 35.56 40.64))
+  (wire (pts (xy 33.02 40.64) (xy 33.02 43.18))
     (stroke (width 0) (type default))
   )
@@
     (stroke (width 0) (type default))
   )
-  (wire (pts (xy 35.56 62.23) (xy 35.56 64.77))
+  (wire (pts (xy 33.02 64.77) (xy 33.02 67.31))
     (stroke (width 0) (type default))
   )
@@
     (stroke (width 0) (type default))
   )
-  (wire (pts (xy 35.56 50.8) (xy 46.99 50.8))
+  (wire (pts (xy 33.02 53.34) (xy 44.45 53.34))
     (stroke (width 0) (type default))
   )
@@
     (effects (font (size 1.27 1.27)) (justify left bottom))
   )
-  (text "Min EN pin input\ncurrent = 2uA" (at 54.61 46.99 0)
+  (text "Min EN pin input\ncurrent = 2uA" (at 52.07 49.53 0)
     (effects (font (size 1.27 1.27)) (justify left bottom))
   )
@@
     (effects (font (size 1.27 1.27)) (justify left bottom))
   )
-  (text "Monitors battery voltage for\nbuck-boost converter.\nVoltage divider calculation\ndone at V_BATT = 3V.\nBuck-boost converter EN shuts off\nat 0.7V.\nV_BATT_BUCK_BOOST_EN = 0.683 \n@ VBATT = 3V"
-    (at 54.61 39.37 0)
+  (text "Monitors battery voltage for\nbuck-boost converter.\nVoltage divider calculation\ndone at V_BATT = 3V.\nBuck-boost converter EN shuts off\nat 0.7V.\n\nV_BATT_BUCK_BOOST_EN = 0.683 \n@ VBATT = 3V\n\nV_BATT_BUCK_BOOST_EN = 0.7\n@ VBATT = 3.075V"
+    (at 52.07 41.91 0)
     (effects (font (size 1.27 1.27)) (justify left bottom))
   )
@@
     )
   )
-  (global_label "BATT_BUCK_BOOST_EN" (shape output) (at 50.8 50.8 0) (fields_autoplaced)
+  (global_label "BATT_BUCK_BOOST_EN" (shape output) (at 48.26 53.34 0) (fields_autoplaced)
     (effects (font (size 1.27 1.27)) (justify left))
-    (property "Intersheetrefs" "${INTERSHEET_REFS}" (at 74.7099 50.8 0)
+    (property "Intersheetrefs" "${INTERSHEET_REFS}" (at 72.1699 53.34 0)
       (effects (font (size 1.27 1.27)) (justify left) hide)
     )
@@
     )
   )
-  (symbol (lib_id "Device:R_US") (at 35.56 57.15 0) (unit 1)
-    (in_bom yes) (on_board yes) (dnp no) (fields_autoplaced)
-    (property "Reference" "R?" (at 38.1 55.88 0)
-      (effects (font (size 1.27 1.27)) (justify left))
-    )
-    (property "Value" "330k" (at 38.1 58.42 0)
-      (effects (font (size 1.27 1.27)) (justify left))
-    )
-    (property "Footprint" "" (at 36.576 57.404 90)
-      (effects (font (size 1.27 1.27)) hide)
-    )
-    (property "Datasheet" "~" (at 35.56 57.15 0)
+  (symbol (lib_id "Device:R_US") (at 33.02 59.69 0) (unit 1)
+    (in_bom yes) (on_board yes) (dnp no) (fields_autoplaced)
+    (property "Reference" "R?" (at 35.56 58.42 0)
+      (effects (font (size 1.27 1.27)) (justify left))
+    )
+    (property "Value" "330k" (at 35.56 60.96 0)
+      (effects (font (size 1.27 1.27)) (justify left))
+    )
+    (property "Footprint" "" (at 34.036 59.944 90)
+      (effects (font (size 1.27 1.27)) hide)
+    )
+    (property "Datasheet" "~" (at 33.02 59.69 0)
       (effects (font (size 1.27 1.27)) hide)
     )
@@
     )
   )
-  (symbol (lib_id "power:GND") (at 35.56 64.77 0) (unit 1)
-    (in_bom yes) (on_board yes) (dnp no) (fields_autoplaced)
-    (property "Reference" "#PWR032" (at 35.56 71.12 0)
-      (effects (font (size 1.27 1.27)) hide)
-    )
-    (property "Value" "GND" (at 35.56 69.85 0)
-      (effects (font (size 1.27 1.27)))
-    )
-    (property "Footprint" "" (at 35.56 64.77 0)
-      (effects (font (size 1.27 1.27)) hide)
-    )
-    (property "Datasheet" "" (at 35.56 64.77 0)
+  (symbol (lib_id "power:GND") (at 33.02 67.31 0) (unit 1)
+    (in_bom yes) (on_board yes) (dnp no) (fields_autoplaced)
+    (property "Reference" "#PWR032" (at 33.02 73.66 0)
+      (effects (font (size 1.27 1.27)) hide)
+    )
+    (property "Value" "GND" (at 33.02 72.39 0)
+      (effects (font (size 1.27 1.27)))
+    )
+    (property "Footprint" "" (at 33.02 67.31 0)
+      (effects (font (size 1.27 1.27)) hide)
+    )
+    (property "Datasheet" "" (at 33.02 67.31 0)
       (effects (font (size 1.27 1.27)) hide)
     )
@@
     )
   )
-  (symbol (lib_id "Device:R_US") (at 35.56 44.45 0) (unit 1)
-    (in_bom yes) (on_board yes) (dnp no) (fields_autoplaced)
-    (property "Reference" "R?" (at 38.1 43.18 0)
-      (effects (font (size 1.27 1.27)) (justify left))
-    )
-    (property "Value" "560k" (at 38.1 45.72 0)
-      (effects (font (size 1.27 1.27)) (justify left))
-    )
-    (property "Footprint" "" (at 36.576 44.704 90)
-      (effects (font (size 1.27 1.27)) hide)
-    )
-    (property "Datasheet" "~" (at 35.56 44.45 0)
+  (symbol (lib_id "Device:R_US") (at 33.02 46.99 0) (unit 1)
+    (in_bom yes) (on_board yes) (dnp no) (fields_autoplaced)
+    (property "Reference" "R?" (at 35.56 45.72 0)
+      (effects (font (size 1.27 1.27)) (justify left))
+    )
+    (property "Value" "560k" (at 35.56 48.26 0)
+      (effects (font (size 1.27 1.27)) (justify left))
+    )
+    (property "Footprint" "" (at 34.036 47.244 90)
+      (effects (font (size 1.27 1.27)) hide)
+    )
+    (property "Datasheet" "~" (at 33.02 46.99 0)
       (effects (font (size 1.27 1.27)) hide)
     )
@@
     )
   )
-  (symbol (lib_id "power:+BATT") (at 35.56 38.1 0) (unit 1)
-    (in_bom yes) (on_board yes) (dnp no) (fields_autoplaced)
-    (property "Reference" "#PWR06" (at 35.56 41.91 0)
-      (effects (font (size 1.27 1.27)) hide)
-    )
-    (property "Value" "+BATT" (at 35.56 33.02 0)
-      (effects (font (size 1.27 1.27)))
-    )
-    (property "Footprint" "" (at 35.56 38.1 0)
-      (effects (font (size 1.27 1.27)) hide)
-    )
-    (property "Datasheet" "" (at 35.56 38.1 0)
+  (symbol (lib_id "power:+BATT") (at 33.02 40.64 0) (unit 1)
+    (in_bom yes) (on_board yes) (dnp no) (fields_autoplaced)
+    (property "Reference" "#PWR06" (at 33.02 44.45 0)
+      (effects (font (size 1.27 1.27)) hide)
+    )
+    (property "Value" "+BATT" (at 33.02 35.56 0)
+      (effects (font (size 1.27 1.27)))
+    )
+    (property "Footprint" "" (at 33.02 40.64 0)
+      (effects (font (size 1.27 1.27)) hide)
+    )
+    (property "Datasheet" "" (at 33.02 40.64 0)
       (effects (font (size 1.27 1.27)) hide)
     )
@@
     )
   )
-  (symbol (lib_id "Device:R_US") (at 46.99 57.15 0) (unit 1)
+  (symbol (lib_id "Device:R_US") (at 44.45 59.69 0) (unit 1)
     (in_bom yes) (on_board yes) (dnp no)
-    (property "Reference" "R?" (at 49.53 55.88 0)
-      (effects (font (size 1.27 1.27)) (justify left))
-    )
-    (property "Value" "330k" (at 49.53 58.42 0)
-      (effects (font (size 1.27 1.27)) (justify left))
-    )
-    (property "Footprint" "" (at 48.006 57.404 90)
-      (effects (font (size 1.27 1.27)) hide)
-    )
-    (property "Datasheet" "~" (at 46.99 57.15 0)
-      (effects (font (size 1.27 1.27)) hide)
-    )
+    (property "Reference" "R?" (at 46.99 58.42 0)
+      (effects (font (size 1.27 1.27)) (justify left))
+    )
+    (property "Value" "330k" (at 46.99 60.96 0)
+      (effects (font (size 1.27 1.27)) (justify left))
+    )
+    (property "Footprint" "" (at 45.466 59.944 90)
+      (effects (font (size 1.27 1.27)) hide)
+    )
+    (property "Datasheet" "~" (at 44.45 59.69 0)
+      (effects (font (size 1.27 1.27)) hide)
+    )

Commit message: continuing to add footprints
Parts:
- C10, C11, C12, C5, C6, C? (x2): footprint (none) -> Capacitor_SMD:C_0805_2012Metric_Pad1.18x1.45mm_HandSolder
- R10, R14, R9, R? (x5): footprint (none) -> Resistor_SMD:R_0805_2012Metric_Pad1.20x1.40mm_HandSolder
Changed lines of the file:
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@@
       (effects (font (size 1.27 1.27)) (justify left))
     )
-    (property "Footprint" "" (at 257.5052 76.2 0)
+    (property "Footprint" "Capacitor_SMD:C_0805_2012Metric_Pad1.18x1.45mm_HandSolder" (at 257.5052 76.2 0)
       (effects (font (size 1.27 1.27)) hide)
     )
@@
       (effects (font (size 1.27 1.27)) (justify left))
     )
-    (property "Footprint" "" (at 83.566 153.924 90)
+    (property "Footprint" "Resistor_SMD:R_0805_2012Metric_Pad1.20x1.40mm_HandSolder" (at 83.566 153.924 90)
       (effects (font (size 1.27 1.27)) hide)
     )
@@
       (effects (font (size 1.27 1.27)) (justify left))
     )
-    (property "Footprint" "" (at 34.036 59.944 90)
+    (property "Footprint" "Resistor_SMD:R_0805_2012Metric_Pad1.20x1.40mm_HandSolder" (at 34.036 59.944 90)
       (effects (font (size 1.27 1.27)) hide)
     )
@@
       (effects (font (size 1.27 1.27)) (justify left))
     )
-    (property "Footprint" "" (at 233.3752 76.2 0)
+    (property "Footprint" "Capacitor_SMD:C_0805_2012Metric_Pad1.18x1.45mm_HandSolder" (at 233.3752 76.2 0)
       (effects (font (size 1.27 1.27)) hide)
     )
@@
       (effects (font (size 1.27 1.27)) (justify left))
     )
-    (property "Footprint" "" (at 31.4452 151.13 0)
+    (property "Footprint" "Capacitor_SMD:C_0805_2012Metric_Pad1.18x1.45mm_HandSolder" (at 31.4452 151.13 0)
       (effects (font (size 1.27 1.27)) hide)
     )
@@
       (effects (font (size 1.27 1.27)) (justify left))
     )
-    (property "Footprint" "" (at 205.486 86.614 90)
+    (property "Footprint" "Resistor_SMD:R_0805_2012Metric_Pad1.20x1.40mm_HandSolder" (at 205.486 86.614 90)
       (effects (font (size 1.27 1.27)) hide)
     )
@@
       (effects (font (size 1.27 1.27)) (justify left))
     )
-    (property "Footprint" "" (at 96.2152 151.13 0)
+    (property "Footprint" "Capacitor_SMD:C_0805_2012Metric_Pad1.18x1.45mm_HandSolder" (at 96.2152 151.13 0)
       (effects (font (size 1.27 1.27)) hide)
     )
@@
       (effects (font (size 1.27 1.27)) (justify left))
     )
-    (property "Footprint" "" (at 103.8352 77.47 0)
+    (property "Footprint" "Capacitor_SMD:C_0805_2012Metric_Pad1.18x1.45mm_HandSolder" (at 103.8352 77.47 0)
       (effects (font (size 1.27 1.27)) hide)
     )
@@
       (effects (font (size 1.27 1.27)) (justify left))
     )
-    (property "Footprint" "" (at 246.0752 76.2 0)
+    (property "Footprint" "Capacitor_SMD:C_0805_2012Metric_Pad1.18x1.45mm_HandSolder" (at 246.0752 76.2 0)
       (effects (font (size 1.27 1.27)) hide)
     )
@@
       (effects (font (size 1.27 1.27)) (justify left))
     )
-    (property "Footprint" "" (at 116.5352 77.47 0)
+    (property "Footprint" "Capacitor_SMD:C_0805_2012Metric_Pad1.18x1.45mm_HandSolder" (at 116.5352 77.47 0)
       (effects (font (size 1.27 1.27)) hide)
     )
@@
       (effects (font (size 1.27 1.27)) (justify left))
     )
-    (property "Footprint" "" (at 129.286 77.724 90)
+    (property "Footprint" "Resistor_SMD:R_0805_2012Metric_Pad1.20x1.40mm_HandSolder" (at 129.286 77.724 90)
       (effects (font (size 1.27 1.27)) hide)
     )
@@
       (effects (font (size 1.27 1.27)) (justify left))
     )
-    (property "Footprint" "" (at 34.036 47.244 90)
+    (property "Footprint" "Resistor_SMD:R_0805_2012Metric_Pad1.20x1.40mm_HandSolder" (at 34.036 47.244 90)
       (effects (font (size 1.27 1.27)) hide)
     )
@@
       (effects (font (size 1.27 1.27)) (justify left))
     )
-    (property "Footprint" "" (at 83.566 166.624 90)
+    (property "Footprint" "Resistor_SMD:R_0805_2012Metric_Pad1.20x1.40mm_HandSolder" (at 83.566 166.624 90)
       (effects (font (size 1.27 1.27)) hide)
     )
@@
       (effects (font (size 1.27 1.27)) (justify left))
     )
-    (property "Footprint" "" (at 205.486 75.184 90)
+    (property "Footprint" "Resistor_SMD:R_0805_2012Metric_Pad1.20x1.40mm_HandSolder" (at 205.486 75.184 90)
       (effects (font (size 1.27 1.27)) hide)
     )
@@
       (effects (font (size 1.27 1.27)) (justify left))
     )
-    (property "Footprint" "" (at 45.466 59.944 90)
-      (effects (font (size 1.27 1.27)) hide)
-    )
+    (property "Footprint" "Resistor_SMD:R_0805_2012Metric_Pad1.20x1.40mm_HandSolder" (at 45.466 59.944 90)
+      (effects (font (size 1.27 1.27)) hide)
+    )
