File: boardlock/testpoints.kicad_sch (KiCad schematic)
At the start: 13 parts

Commit message: name change
Parts:
- TP5: value RX -> UART_RX
- TP6: value TX -> UART_TX
Connections:
- net M_RX renamed M_UART_RX
- net M_TX renamed M_UART_TX
Changed lines of the file:
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@@
     )
   )
-  (global_label "M_RX" (shape input) (at 73.66 22.86 180) (fields_autoplaced)
-    (effects (font (size 1.27 1.27)) (justify right))
-    (property "Intersheetrefs" "${INTERSHEET_REFS}" (at 65.7763 22.86 0)
+  (global_label "M_UART_RX" (shape input) (at 73.66 22.86 180) (fields_autoplaced)
+    (effects (font (size 1.27 1.27)) (justify right))
+    (property "Intersheetrefs" "${INTERSHEET_REFS}" (at 60.152 22.86 0)
       (effects (font (size 1.27 1.27)) (justify right) hide)
     )
@@
     )
   )
-  (global_label "M_TX" (shape input) (at 73.66 26.67 180) (fields_autoplaced)
-    (effects (font (size 1.27 1.27)) (justify right))
-    (property "Intersheetrefs" "${INTERSHEET_REFS}" (at 66.0787 26.67 0)
+  (global_label "M_UART_TX" (shape input) (at 73.66 26.67 180) (fields_autoplaced)
+    (effects (font (size 1.27 1.27)) (justify right))
+    (property "Intersheetrefs" "${INTERSHEET_REFS}" (at 60.4544 26.67 0)
       (effects (font (size 1.27 1.27)) (justify right) hide)
     )
@@
       (effects (font (size 1.27 1.27)))
     )
-    (property "Value" "TX" (at 87.63 26.67 90)
+    (property "Value" "UART_TX" (at 87.63 26.67 90)
       (effects (font (size 1.27 1.27)))
     )
@@
       (effects (font (size 1.27 1.27)))
     )
-    (property "Value" "RX" (at 87.63 22.86 90)
-      (effects (font (size 1.27 1.27)))
-    )
+    (property "Value" "UART_RX" (at 87.63 22.86 90)
+      (effects (font (size 1.27 1.27)))
+    )
