File: boardlock/audio.kicad_sch (KiCad schematic)
At the start: 20 parts, among them J3 5033981892, Q2 MMBT4401, Q4 BSS84PWH6327XTSA1, U7 MAX98357AETE+T

Commit message: footprint work
Parts:
- Q2: footprint (none) -> Package_TO_SOT_SMD:SOT-23-3
- gave numbers to parts that had none: 11
Changed lines of the file:
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@@
         )
         (path "/e1fc29ce-837e-4062-84d8-c7e423f9eab9/1eb676fb-9e7a-4e01-ba1e-2eff94d7b66e"
-          (reference "Q?") (unit 1)
+          (reference "Q8") (unit 1)
         )
       )
@@
   (symbol (lib_id "Connector_Generic:Conn_01x02") (at 203.2 55.88 0) (unit 1)
     (in_bom yes) (on_board yes) (dnp no) (fields_autoplaced)
-    (property "Reference" "J?" (at 205.74 55.88 0)
+    (property "Reference" "J4" (at 205.74 55.88 0)
       (effects (font (size 1.27 1.27)) (justify left))
     )
@@
       (project "boardlock"
         (path "/e1fc29ce-837e-4062-84d8-c7e423f9eab9/1eb676fb-9e7a-4e01-ba1e-2eff94d7b66e"
-          (reference "J?") (unit 1)
+          (reference "J4") (unit 1)
         )
       )
@@
   (symbol (lib_id "Device:C") (at 147.32 67.31 0) (unit 1)
     (in_bom yes) (on_board yes) (dnp no) (fields_autoplaced)
-    (property "Reference" "C?" (at 150.241 66.0979 0)
+    (property "Reference" "C32" (at 150.241 66.0979 0)
       (effects (font (size 1.27 1.27)) (justify left))
     )
@@
       (project "boardlock"
         (path "/e1fc29ce-837e-4062-84d8-c7e423f9eab9/1eb676fb-9e7a-4e01-ba1e-2eff94d7b66e"
-          (reference "C?") (unit 1)
+          (reference "C32") (unit 1)
         )
       )
@@
   (symbol (lib_id "Connector_Generic:Conn_01x02") (at 246.38 124.46 0) (unit 1)
     (in_bom yes) (on_board yes) (dnp no) (fields_autoplaced)
-    (property "Reference" "J?" (at 248.92 124.46 0)
+    (property "Reference" "J5" (at 248.92 124.46 0)
       (effects (font (size 1.27 1.27)) (justify left))
     )
@@
       (project "boardlock"
         (path "/e1fc29ce-837e-4062-84d8-c7e423f9eab9/1eb676fb-9e7a-4e01-ba1e-2eff94d7b66e"
-          (reference "J?") (unit 1)
+          (reference "J5") (unit 1)
         )
       )
@@
   (symbol (lib_id "Device:C") (at 62.23 44.45 0) (unit 1)
     (in_bom yes) (on_board yes) (dnp no) (fields_autoplaced)
-    (property "Reference" "C?" (at 65.151 43.2379 0)
+    (property "Reference" "C30" (at 65.151 43.2379 0)
       (effects (font (size 1.27 1.27)) (justify left))
     )
@@
       (project "boardlock"
         (path "/e1fc29ce-837e-4062-84d8-c7e423f9eab9/1eb676fb-9e7a-4e01-ba1e-2eff94d7b66e"
-          (reference "C?") (unit 1)
+          (reference "C30") (unit 1)
         )
       )
@@
   (symbol (lib_id "Device:FerriteBead_Small") (at 140.97 53.34 270) (unit 1)
     (in_bom yes) (on_board yes) (dnp no)
-    (property "Reference" "FB?" (at 140.97 46.99 90)
+    (property "Reference" "FB1" (at 140.97 46.99 90)
       (effects (font (size 1.27 1.27)))
     )
@@
       (project "boardlock"
         (path "/e1fc29ce-837e-4062-84d8-c7e423f9eab9/1eb676fb-9e7a-4e01-ba1e-2eff94d7b66e"
-          (reference "FB?") (unit 1)
+          (reference "FB1") (unit 1)
         )
       )
@@
   (symbol (lib_id "Device:FerriteBead_Small") (at 140.97 60.96 270) (unit 1)
     (in_bom yes) (on_board yes) (dnp no)
-    (property "Reference" "FB?" (at 140.97 67.31 90)
+    (property "Reference" "FB2" (at 140.97 67.31 90)
       (effects (font (size 1.27 1.27)))
     )
@@
       (project "boardlock"
         (path "/e1fc29ce-837e-4062-84d8-c7e423f9eab9/1eb676fb-9e7a-4e01-ba1e-2eff94d7b66e"
-          (reference "FB?") (unit 1)
+          (reference "FB2") (unit 1)
         )
       )
@@
   (symbol (lib_id "Device:R_US") (at 22.86 52.07 0) (unit 1)
     (in_bom yes) (on_board yes) (dnp no)
-    (property "Reference" "R?" (at 20.32 50.8 0)
+    (property "Reference" "R57" (at 20.32 50.8 0)
       (effects (font (size 1.27 1.27)) (justify right))
     )
@@
       (project "boardlock"
         (path "/e1fc29ce-837e-4062-84d8-c7e423f9eab9/1eb676fb-9e7a-4e01-ba1e-2eff94d7b66e"
-          (reference "R?") (unit 1)
+          (reference "R57") (unit 1)
         )
       )
@@
   (symbol (lib_id "Device:C") (at 166.37 57.15 0) (unit 1)
     (in_bom yes) (on_board yes) (dnp no) (fields_autoplaced)
-    (property "Reference" "C?" (at 169.291 55.9379 0)
+    (property "Reference" "C31" (at 169.291 55.9379 0)
       (effects (font (size 1.27 1.27)) (justify left))
     )
@@
       (project "boardlock"
         (path "/e1fc29ce-837e-4062-84d8-c7e423f9eab9/1eb676fb-9e7a-4e01-ba1e-2eff94d7b66e"
-          (reference "C?") (unit 1)
+          (reference "C31") (unit 1)
         )
       )
@@
         )
         (path "/e1fc29ce-837e-4062-84d8-c7e423f9eab9/1eb676fb-9e7a-4e01-ba1e-2eff94d7b66e"
-          (reference "R?") (unit 1)
+          (reference "R59") (unit 1)
         )
       )
@@
   (symbol (lib_id "Device:C") (at 160.02 67.31 0) (unit 1)
     (in_bom yes) (on_board yes) (dnp no) (fields_autoplaced)
-    (property "Reference" "C?" (at 162.941 66.0979 0)
+    (property "Reference" "C33" (at 162.941 66.0979 0)
       (effects (font (size 1.27 1.27)) (justify left))
     )
@@
       (project "boardlock"
         (path "/e1fc29ce-837e-4062-84d8-c7e423f9eab9/1eb676fb-9e7a-4e01-ba1e-2eff94d7b66e"
-          (reference "C?") (unit 1)
+          (reference "C33") (unit 1)
         )
       )
@@
   (symbol (lib_id "Device:R_US") (at 69.85 67.31 0) (unit 1)
     (in_bom yes) (on_board yes) (dnp no)
-    (property "Reference" "R?" (at 67.31 66.04 0)
+    (property "Reference" "R58" (at 67.31 66.04 0)
       (effects (font (size 1.27 1.27)) (justify right))
     )
@@
       (project "boardlock"
         (path "/e1fc29ce-837e-4062-84d8-c7e423f9eab9/1eb676fb-9e7a-4e01-ba1e-2eff94d7b66e"
-          (reference "R?") (unit 1)
+          (reference "R58") (unit 1)
         )
       )
@@
         )
         (path "/e1fc29ce-837e-4062-84d8-c7e423f9eab9/1eb676fb-9e7a-4e01-ba1e-2eff94d7b66e"
-          (reference "R?") (unit 1)
+          (reference "R61") (unit 1)
         )
       )
@@
   (symbol (lib_id "Device:R_US") (at 22.86 41.91 0) (unit 1)
     (in_bom yes) (on_board yes) (dnp no)
-    (property "Reference" "R?" (at 20.32 40.64 0)
+    (property "Reference" "R56" (at 20.32 40.64 0)
       (effects (font (size 1.27 1.27)) (justify right))
     )
@@
       (project "boardlock"
         (path "/e1fc29ce-837e-4062-84d8-c7e423f9eab9/1eb676fb-9e7a-4e01-ba1e-2eff94d7b66e"
-          (reference "R?") (unit 1)
+          (reference "R56") (unit 1)
         )
       )
@@
         )
         (path "/e1fc29ce-837e-4062-84d8-c7e423f9eab9/1eb676fb-9e7a-4e01-ba1e-2eff94d7b66e"
-          (reference "R?") (unit 1)
+          (reference "R60") (unit 1)
         )
       )
@@
       (effects (font (size 1.27 1.27)) (justify left))
     )
-    (property "Footprint" "" (at 207.01 116.84 0)
+    (property "Footprint" "Package_TO_SOT_SMD:SOT-23-3" (at 207.01 116.84 0)
       (effects (font (size 1.27 1.27)) hide)
     )
@@
         )
         (path "/e1fc29ce-837e-4062-84d8-c7e423f9eab9/1eb676fb-9e7a-4e01-ba1e-2eff94d7b66e"
-          (reference "Q?") (unit 1)
-        )
-      )
+          (reference "Q9") (unit 1)
+        )
+      )

Commit message: changes
Changed lines of the file:
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@@
   )
   (text "Channel Selection\nLEFT = VDD (0 Ohm)\nRIGHT = (94*VDD - 100) kOhm\nL/R = (22.2*VDD-100) kOhm\n\nMight be not needed since\nI got this work without\nthe signal being connected."
-    (at 41.91 93.98 0)
+    (at 41.91 97.79 0)
     (effects (font (size 1.27 1.27)) (justify left bottom))
   )
