File: boardlock/battery.kicad_sch (KiCad schematic)
At the start: 18 parts, among them J2 Conn_01x02_MountingPin, U4 BQ27441DRZR-G1A, U5 BQ24075RGT

Commit message: more Zecong edits
Connections:
- net V_USB renamed VBUS
Changed lines of the file:
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@@
   (junction (at 196.85 125.73) (diameter 0) (color 0 0 0 0)
   )
+  (junction (at 58.42 66.04) (diameter 0) (color 0 0 0 0)
+  )
+  (junction (at 184.15 130.81) (diameter 0) (color 0 0 0 0)
+  )
+  (junction (at 179.07 135.89) (diameter 0) (color 0 0 0 0)
+  )
+  (junction (at 189.23 26.67) (diameter 0) (color 0 0 0 0)
+  )
+  (junction (at 58.42 81.28) (diameter 0) (color 0 0 0 0)
+  )
+  (junction (at 184.15 135.89) (diameter 0) (color 0 0 0 0)
+  )
+  (junction (at 121.92 97.79) (diameter 0) (color 0 0 0 0)
+  )
+  (junction (at 59.69 151.13) (diameter 0) (color 0 0 0 0)
+  )
   (junction (at 83.82 45.72) (diameter 0) (color 0 0 0 0)
   )
-  (junction (at 58.42 66.04) (diameter 0) (color 0 0 0 0)
-  )
-  (junction (at 184.15 130.81) (diameter 0) (color 0 0 0 0)
-  )
-  (junction (at 179.07 135.89) (diameter 0) (color 0 0 0 0)
-  )
-  (junction (at 189.23 26.67) (diameter 0) (color 0 0 0 0)
-  )
-  (junction (at 58.42 81.28) (diameter 0) (color 0 0 0 0)
-  )
-  (junction (at 184.15 135.89) (diameter 0) (color 0 0 0 0)
-  )
-  (junction (at 121.92 97.79) (diameter 0) (color 0 0 0 0)
-  )
-  (junction (at 59.69 151.13) (diameter 0) (color 0 0 0 0)
-  )
   (junction (at 213.36 152.4) (diameter 0) (color 0 0 0 0)
   )
@@
     (stroke (width 0) (type default))
   )
-  (wire (pts (xy 73.66 45.72) (xy 83.82 45.72))
-    (stroke (width 0) (type default))
-  )
   (wire (pts (xy 189.23 48.26) (xy 207.01 48.26))
     (stroke (width 0) (type default))
@@
   )
   (wire (pts (xy 231.14 125.73) (xy 234.95 125.73))
+    (stroke (width 0) (type default))
+  )
+  (wire (pts (xy 83.82 40.64) (xy 83.82 45.72))
     (stroke (width 0) (type default))
   )
@@
     (property "Intersheetrefs" "${INTERSHEET_REFS}" (at 130.7713 73.66 0)
       (effects (font (size 1.27 1.27)) (justify left) hide)
-    )
-  )
-  (global_label "V_USB" (shape input) (at 73.66 45.72 180) (fields_autoplaced)
-    (effects (font (size 1.27 1.27)) (justify right))
-    (property "Intersheetrefs" "${INTERSHEET_REFS}" (at 64.8086 45.72 0)
-      (effects (font (size 1.27 1.27)) (justify right) hide)
     )
   )
@@
         )
       )
+    )
+  )
+  (symbol (lib_id "power:VBUS") (at 83.82 40.64 0) (unit 1)
+    (in_bom yes) (on_board yes) (dnp no) (fields_autoplaced)
+    (property "Reference" "#PWR064" (at 83.82 44.45 0)
+      (effects (font (size 1.27 1.27)) hide)
+    )
+    (property "Value" "VBUS" (at 83.82 35.56 0)
+      (effects (font (size 1.27 1.27)))
+    )
+    (property "Footprint" "" (at 83.82 40.64 0)
+      (effects (font (size 1.27 1.27)) hide)
+    )
+    (property "Datasheet" "" (at 83.82 40.64 0)
+      (effects (font (size 1.27 1.27)) hide)
+    )
+    (pin "1")
+    (instances
+      (project "boardlock"
+        (path "/e1fc29ce-837e-4062-84d8-c7e423f9eab9/a05f4dcd-7a18-4529-a05e-43353e81fbf8"
+          (reference "#PWR064") (unit 1)
+        )
+      )

Commit message: lab updates
Other:
- note removed: "Need to add to micro sheet"
Changed lines of the file:
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@@
     (effects (font (size 5 5) (thickness 1) bold) (justify left bottom))
-  )
-  (text "Need to add to \nmicro sheet" (at 234.95 124.46 0)
-    (effects (font (size 1.27 1.27)) (justify left bottom))
   )
   (text "+Batt is the battery\nvoltage after the\ncoloumb shunt resistor"
