File: boardlock/sensors.kicad_sch (KiCad schematic)
At the start: 16 parts, among them Q2 Q_NPN_BCE, Q3 Q_NPN_BCE, Q4 BSS84PWH6327XTSA1, U1 LSM6DSO32, U3 SAM-M8Q

Commit message: NPN?
Parts:
- removed Q3: Q_NPN_BCE, symbol Device:Q_NPN_BCE
- removed R5: R_US, symbol Device:R_US
Connections:
- net M_IMU_POWER: now also Q4.1 (G), R6.2
Other:
- note added: "LOOK AT LATER"
- note added: "THIS NEEDS TO CHANGE"
Changed lines of the file:
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@@
-    (stroke (width 0) (type default))
-  )
-  (wire (pts (xy 67.31 77.47) (xy 67.31 83.82))
     (stroke (width 0) (type default))
   )
@@
     (stroke (width 0) (type default))
   )
-  (wire (pts (xy 55.88 72.39) (xy 59.69 72.39))
+  (wire (pts (xy 62.23 64.77) (xy 67.31 64.77))
     (stroke (width 0) (type default))
   )
@@
     (stroke (width 0) (type default))
   )
-  (wire (pts (xy 67.31 64.77) (xy 67.31 67.31))
-    (stroke (width 0) (type default))
-  )
   (wire (pts (xy 210.82 104.14) (xy 210.82 106.68))
     (stroke (width 0) (type default))
@@
   )
   (wire (pts (xy 212.09 50.8) (xy 212.09 53.34))
-    (stroke (width 0) (type default))
-  )
-  (wire (pts (xy 43.18 72.39) (xy 48.26 72.39))
     (stroke (width 0) (type default))
   )
@@
     (at 154.94 92.71 0)
     (effects (font (size 1.27 1.27)) (justify left bottom))
+  )
+  (text "THIS NEEDS TO CHANGE" (at 215.9 67.31 0)
+    (effects (font (size 1.27 1.27) (thickness 0.254) bold) (justify left bottom))
   )
   (text "IMU Power Saving Circuit" (at 34.29 48.26 0)
@@
   (text "SDO/SAO (Z) \nDetermines I2C Addr.\n0110101(Z) b\n" (at 27.94 177.8 0)
     (effects (font (size 2.5 2.5)) (justify left bottom))
+  )
+  (text "LOOK AT LATER" (at 64.77 72.39 0)
+    (effects (font (size 1.27 1.27) bold) (justify left bottom))
   )
   (text "NOTE TO SELF: check which wires do and do not need resistors\n"
@@
     )
   )
-  (global_label "M_IMU_POWER" (shape input) (at 43.18 72.39 180) (fields_autoplaced)
+  (global_label "M_IMU_POWER" (shape input) (at 62.23 64.77 180) (fields_autoplaced)
     (effects (font (size 1.27 1.27)) (justify right))
-    (property "Intersheetrefs" "${INTERSHEET_REFS}" (at 26.9506 72.39 0)
+    (property "Intersheetrefs" "${INTERSHEET_REFS}" (at 46.0006 64.77 0)
       (effects (font (size 1.27 1.27)) (justify right) hide)
     )
@@
         (path "/e1fc29ce-837e-4062-84d8-c7e423f9eab9/a4a6f965-a4d9-4da6-b64e-79eda0daabe5"
           (reference "#PWR07") (unit 1)
-        )
-      )
-    )
-  )
-  (symbol (lib_id "power:GND") (at 67.31 83.82 0) (unit 1)
-    (in_bom yes) (on_board yes) (dnp no) (fields_autoplaced)
-    (property "Reference" "#PWR06" (at 67.31 90.17 0)
-      (effects (font (size 1.27 1.27)) hide)
-    )
-    (property "Value" "GND" (at 67.31 87.9531 0)
-      (effects (font (size 1.27 1.27)))
-    )
-    (property "Footprint" "" (at 67.31 83.82 0)
-      (effects (font (size 1.27 1.27)) hide)
-    )
-    (property "Datasheet" "" (at 67.31 83.82 0)
-      (effects (font (size 1.27 1.27)) hide)
-    )
-    (pin "1")
-    (instances
-      (project "boardlock"
-        (path "/48f24f42-fd64-4860-9f12-ca34cf195758/17b4aebf-aea4-4bb2-a07c-86de8cf47820"
-          (reference "#PWR06") (unit 1)
-        )
-        (path "/48f24f42-fd64-4860-9f12-ca34cf195758/17b4aebf-aea4-4bb2-a07c-86de8cf47820/50767468-7b8a-48f0-9e61-53ec0e447e69"
-          (reference "#PWR06") (unit 1)
-        )
-      )
-      (project "boardlock"
-        (path "/e1fc29ce-837e-4062-84d8-c7e423f9eab9/a4a6f965-a4d9-4da6-b64e-79eda0daabe5"
-          (reference "#PWR06") (unit 1)
         )
       )
@@
     )
   )
-  (symbol (lib_id "Device:R_US") (at 52.07 72.39 90) (unit 1)
-    (in_bom yes) (on_board yes) (dnp no) (fields_autoplaced)
-    (property "Reference" "R5" (at 52.07 67.3567 90)
-      (effects (font (size 1.27 1.27)))
-    )
-    (property "Value" "R_US" (at 52.07 69.7809 90)
-      (effects (font (size 1.27 1.27)))
-    )
-    (property "Footprint" "" (at 52.324 71.374 90)
-      (effects (font (size 1.27 1.27)) hide)
-    )
-    (property "Datasheet" "~" (at 52.07 72.39 0)
-      (effects (font (size 1.27 1.27)) hide)
-    )
-    (pin "1")
-    (pin "2")
-    (instances
-      (project "boardlock"
-        (path "/48f24f42-fd64-4860-9f12-ca34cf195758/17b4aebf-aea4-4bb2-a07c-86de8cf47820"
-          (reference "R5") (unit 1)
-        )
-        (path "/48f24f42-fd64-4860-9f12-ca34cf195758/17b4aebf-aea4-4bb2-a07c-86de8cf47820/50767468-7b8a-48f0-9e61-53ec0e447e69"
-          (reference "R5") (unit 1)
-        )
-      )
-      (project "boardlock"
-        (path "/e1fc29ce-837e-4062-84d8-c7e423f9eab9/a4a6f965-a4d9-4da6-b64e-79eda0daabe5"
-          (reference "R1") (unit 1)
-        )
-      )
-    )
-  )
   (symbol (lib_id "Device:R_US") (at 55.88 140.97 90) (unit 1)
     (in_bom yes) (on_board yes) (dnp no) (fields_autoplaced)
@@
         )
       )
-    )
-  )
-  (symbol (lib_id "Device:Q_NPN_BCE") (at 64.77 72.39 0) (unit 1)
-    (in_bom yes) (on_board yes) (dnp no) (fields_autoplaced)
-    (property "Reference" "Q3" (at 69.6214 71.1779 0)
-      (effects (font (size 1.27 1.27)) (justify left))
-    )
-    (property "Value" "Q_NPN_BCE" (at 69.6214 73.6021 0)
-      (effects (font (size 1.27 1.27)) (justify left))
-    )
-    (property "Footprint" "" (at 69.85 69.85 0)
-      (effects (font (size 1.27 1.27)) hide)
-    )
-    (property "Datasheet" "~" (at 64.77 72.39 0)
-      (effects (font (size 1.27 1.27)) hide)
-    )
-    (pin "1")
-    (pin "2")
-    (pin "3")
-    (instances
-      (project "boardlock"
-        (path "/48f24f42-fd64-4860-9f12-ca34cf195758/17b4aebf-aea4-4bb2-a07c-86de8cf47820"
-          (reference "Q3") (unit 1)
-        )
-        (path "/48f24f42-fd64-4860-9f12-ca34cf195758/17b4aebf-aea4-4bb2-a07c-86de8cf47820/50767468-7b8a-48f0-9e61-53ec0e447e69"
-          (reference "Q3") (unit 1)
-        )
-      )
-      (project "boardlock"
-        (path "/e1fc29ce-837e-4062-84d8-c7e423f9eab9/a4a6f965-a4d9-4da6-b64e-79eda0daabe5"
-          (reference "Q1") (unit 1)
-        )
-      )

Commit message: More zecong edits
Other:
- company: (none) -> Schetmatic
- title: (none) -> BoardLock Schematic
Changed lines of the file:
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@@
 (kicad_sch (version 20230121) (generator eeschema)
   (paper "A4")
+  (title_block
+    (title "BoardLock Schematic")
+    (rev "Rev1")
+    (company "Schetmatic")
+  )
   (junction (at 67.31 52.07) (diameter 0) (color 0 0 0 0)
   )

Commit message: gps updates and protocol testpoints
Parts:
- removed R6: R_US, symbol Device:R_US
- added BT1: Battery, symbol Device:Battery
- added C21: C_Small, symbol Device:C_Small
- added D1: 0.5A/40V/420mV, symbol Device:D_Schottky
- added Q2: MMBT4401, symbol Device:Q_NPN_BCE
- added R10, R9: 470, symbol Device:R_US
- added R7, R8: R_US, symbol Device:R_US
- added R9: 3.3k, symbol Device:R_US
- added TP1: TIMEPULSE, symbol Connector:TestPoint
- added TP15: GPS_POWER, symbol Connector:TestPoint
- added TP16: IMU_POWER, symbol Connector:TestPoint
- added TP2: GPS_RESET_N, symbol Connector:TestPoint
- added TP3: GPS_SAFE_N, symbol Connector:TestPoint
- added TP4: GPS_EXTINT, symbol Connector:TestPoint
- added TP9: IMU_INT2, symbol Connector:TestPoint
- Q2: value Q_NPN_BCE -> MMBT4401
- R10, R9: value R_US -> 22
Connections:
- net +3V3: now also R7.1
- net GND: now also BT1.2 (-), C21.2, Q2.3 (E)
- net GPS_POWER: now also Q4.3 (D), D1.2 (A)
- net IMU_POWER: no longer Q4.3 (D)
- net M_GPS_EXTINT: now also TP4.1
- net M_GPS_POWER: now also TP15.1
- net M_IMU_INT2: now also TP9.1
- net M_IMU_POWER: now also R8.1, TP16.1; no longer Q4.1 (G)
- net at U3.13 (TXD): now also R10.2
- net at U3.14 (RXD): now also R9.2
- net at U3.18 (~{RESET}): now also TP2.1
- net at U3.7 (TIMEPULSE): now also TP1.1
- net at U3.8 (~{SAFEBOOT}): now also TP3.1
- new net: Q2.1 (B), R8.2
- new net: Q2.2 (C), Q4.1 (G), R7.2
- new net: D1.1 (K), R9.2
- new net BACKUP: BT1.1 (+), C21.1, R9.1
- new net M_RX: R10.1
- new net M_TX: R9.1
- no-connect marks 4 -> 1
Other:
- note added: "Battery Initial Charge: 2.3-2.8V Battery Charge Rate: 1mA MAX Voff: 2.0V 72 hours charge time from 2.0-3.1V"
- note added: "From https://cdn.sparkfun.com/assets/0/b/0/6/7/SparkFun_Ublox_SAM-M8Q_V10.pdf?_gl= 1*61f7uk*_ga*MTY1MzIxMzcxNy4xNjkzMzIxMDQy*_ga_T369JS7J9N*MTY5NTc0MzczNi41LjEuMTY5NTc0Mzc1OS4zNy4wLjA."
- note added: "KEEP?"
- note added: "TODO"
- note removed: "LOOK AT LATER"
- note removed: "THIS NEEDS TO CHANGE"
- moved on the sheet: Q2, Q4, R10, R7, R8, R9

Commit message: imu check
Parts:
- added C22: 1.0uF, symbol Device:C_Small
- added TP21: IMU_INT1, symbol Connector:TestPoint
- C21: value C_Small -> 1.0uF
Connections:
- net GND: now also C22.2
- net GPS_POWER: now also C22.1
- net at U1.4 (INT1): now also TP21.1
- no-connect marks 1 -> 0
Other:
- note added: "From https://cdn.sparkfun.com/assets/0/b/0/6/7/ SparkFun_Ublox_SAM-M8Q_V10.pdf?_gl= 1*61f7uk*_ga*MTY1MzIxMzcxNy4xNjkzMzIxMDQy*_ga_ T369JS7J9N*MTY5NTc0MzczNi41LjEuMTY5NTc0Mzc1OS4zNy4wLjA."
- note added: "ceramic"
- note added: "mode 1 because we don't need it to be I2C master"
- note removed: "NOTE TO SELF: check which wires do and do not need resistors"
Changed lines of the file:
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@@
   (junction (at 62.23 124.46) (diameter 0) (color 0 0 0 0)
   )
-  (no_connect (at 104.14 130.81))
   (wire (pts (xy 199.39 116.84) (xy 200.66 116.84))
     (stroke (width 0) (type default))
@@
     (stroke (width 0) (type default))
   )
+  (wire (pts (xy 276.86 130.81) (xy 276.86 132.08))
+    (stroke (width 0) (type default))
+  )
   (wire (pts (xy 212.09 154.94) (xy 213.36 154.94))
     (stroke (width 0) (type default))
@@
     (stroke (width 0) (type default))
   )
+  (wire (pts (xy 276.86 124.46) (xy 276.86 125.73))
+    (stroke (width 0) (type default))
+  )
   (wire (pts (xy 74.93 114.3) (xy 74.93 110.49))
     (stroke (width 0) (type default))
@@
   )
   (wire (pts (xy 226.06 114.3) (xy 237.49 114.3))
+    (stroke (width 0) (type default))
+  )
+  (wire (pts (xy 104.14 130.81) (xy 105.41 130.81))
     (stroke (width 0) (type default))
   )
@@
   (text "TIMEPULSE (Output)\nConfigurable Timepulse\nsignal (Default 1Hz).\nLeave open if not used."
     (at 154.94 92.71 0)
+    (effects (font (size 1.27 1.27)) (justify left bottom))
+  )
+  (text "ceramic" (at 64.77 121.92 0)
     (effects (font (size 1.27 1.27)) (justify left bottom))
   )
@@
     (effects (font (size 2.5 2.5) (thickness 0.5) bold) (justify left bottom))
   )
+  (text "From https://cdn.sparkfun.com/assets/0/b/0/6/7/\nSparkFun_Ublox_SAM-M8Q_V10.pdf?_gl=\n1*61f7uk*_ga*MTY1MzIxMzcxNy4xNjkzMzIxMDQy*_ga_\nT369JS7J9N*MTY5NTc0MzczNi41LjEuMTY5NTc0Mzc1OS4zNy4wLjA."
+    (at 260.35 119.38 0)
+    (effects (font (size 0.5 0.5)) (justify left bottom))
+  )
   (text "GPS Module" (at 191.77 91.44 0)
     (effects (font (size 1.27 1.27)) (justify left bottom))
   )
   (text "Q: Are these resistors the R>20ohm \nresistors that are used to avoid \ninterference discussed in 1.6 of \nHardwareIntegrationManual?"
-    (at 238.76 143.51 0)
+    (at 228.6 137.16 0)
     (effects (font (size 1.27 1.27)) (justify left bottom))
   )
@@
     (effects (font (size 0.5 0.5)) (justify left bottom))
   )
-  (text "NOTE TO SELF: check which wires do and do not need resistors\n"
-    (at 53.34 187.96 0)
-    (effects (font (size 1.27 1.27) (thickness 0.254) bold) (justify left bottom))
+  (text "ceramic" (at 77.47 121.92 0)
+    (effects (font (size 1.27 1.27)) (justify left bottom))
+  )
+  (text "mode 1 because we don't \nneed it to be I2C master" (at 19.05 102.87 0)
+    (effects (font (size 1.27 1.27)) (justify left bottom))
   )
   (text "TODO\n" (at 214.63 105.41 0)
@@
   (label "BACKUP" (at 276.86 59.69 0) (fields_autoplaced)
     (effects (font (size 1.27 1.27)) (justify left bottom))
+  )
+  (label "GPS_POWER" (at 276.86 124.46 180) (fields_autoplaced)
+    (effects (font (size 1.27 1.27)) (justify right bottom))
   )
   (label "IMU_POWER" (at 71.12 146.05 180) (fields_autoplaced)
@@
     )
   )
+  (symbol (lib_id "Device:C_Small") (at 276.86 128.27 0) (unit 1)
+    (in_bom yes) (on_board yes) (dnp no) (fields_autoplaced)
+    (property "Reference" "C22" (at 279.4 127.0063 0)
+      (effects (font (size 1.27 1.27)) (justify left))
+    )
+    (property "Value" "1.0uF" (at 279.4 129.5463 0)
+      (effects (font (size 1.27 1.27)) (justify left))
+    )
+    (property "Footprint" "" (at 276.86 128.27 0)
+      (effects (font (size 1.27 1.27)) hide)
+    )
+    (property "Datasheet" "~" (at 276.86 128.27 0)
+      (effects (font (size 1.27 1.27)) hide)
+    )
+    (pin "1")
+    (pin "2")
+    (instances
+      (project "boardlock"
+        (path "/e1fc29ce-837e-4062-84d8-c7e423f9eab9/a4a6f965-a4d9-4da6-b64e-79eda0daabe5"
+          (reference "C22") (unit 1)
+        )
+      )
+    )
+  )
   (symbol (lib_id "Connector:TestPoint") (at 199.39 121.92 90) (unit 1)
     (in_bom yes) (on_board yes) (dnp no)
@@
         (path "/e1fc29ce-837e-4062-84d8-c7e423f9eab9/a4a6f965-a4d9-4da6-b64e-79eda0daabe5"
           (reference "TP2") (unit 1)
+        )
+      )
+    )
+  )
+  (symbol (lib_id "Connector:TestPoint") (at 105.41 130.81 270) (unit 1)
+    (in_bom yes) (on_board yes) (dnp no)
+    (property "Reference" "TP21" (at 123.19 130.81 90)
+      (effects (font (size 1.27 1.27)))
+    )
+    (property "Value" "IMU_INT1" (at 115.57 130.81 90)
+      (effects (font (size 1.27 1.27)))
+    )
+    (property "Footprint" "" (at 105.41 135.89 0)
+      (effects (font (size 1.27 1.27)) hide)
+    )
+    (property "Datasheet" "~" (at 105.41 135.89 0)
+      (effects (font (size 1.27 1.27)) hide)
+    )
+    (pin "1")
+    (instances
+      (project "boardlock"
+        (path "/e1fc29ce-837e-4062-84d8-c7e423f9eab9/a4a6f965-a4d9-4da6-b64e-79eda0daabe5"
+          (reference "TP21") (unit 1)
         )
       )
@@
     )
   )
+  (symbol (lib_id "power:GND") (at 276.86 132.08 0) (unit 1)
+    (in_bom yes) (on_board yes) (dnp no) (fields_autoplaced)
+    (property "Reference" "#PWR01" (at 276.86 138.43 0)
+      (effects (font (size 1.27 1.27)) hide)
+    )
+    (property "Value" "GND" (at 276.86 136.2131 0)
+      (effects (font (size 1.27 1.27)))
+    )
+    (property "Footprint" "" (at 276.86 132.08 0)
+      (effects (font (size 1.27 1.27)) hide)
+    )
+    (property "Datasheet" "" (at 276.86 132.08 0)
+      (effects (font (size 1.27 1.27)) hide)
+    )
+    (pin "1")
+    (instances
+      (project "boardlock"
+        (path "/48f24f42-fd64-4860-9f12-ca34cf195758/17b4aebf-aea4-4bb2-a07c-86de8cf47820"
+          (reference "#PWR01") (unit 1)
+        )
+      )
+      (project "boardlock"
+        (path "/e1fc29ce-837e-4062-84d8-c7e423f9eab9/a4a6f965-a4d9-4da6-b64e-79eda0daabe5"
+          (reference "#PWR062") (unit 1)
+        )
+      )
+    )
+  )
   (symbol (lib_id "power:GND") (at 274.32 72.39 0) (unit 1)
     (in_bom yes) (on_board yes) (dnp no) (fields_autoplaced)
@@
       (effects (font (size 1.27 1.27)) (justify left))
     )
-    (property "Value" "C_Small" (at 276.86 67.3163 0)
-      (effects (font (size 1.27 1.27)) (justify left))
-    )
+    (property "Value" "1.0uF" (at 276.86 67.3163 0)
+      (effects (font (size 1.27 1.27)) (justify left))
+    )

Commit message: name change
Connections:
- net M_RX renamed M_UART_RX
- net M_TX renamed M_UART_TX
Changed lines of the file:
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@@
   )
   (text "From https://cdn.sparkfun.com/assets/0/b/0/6/7/\nSparkFun_Ublox_SAM-M8Q_V10.pdf?_gl=\n1*61f7uk*_ga*MTY1MzIxMzcxNy4xNjkzMzIxMDQy*_ga_\nT369JS7J9N*MTY5NTc0MzczNi41LjEuMTY5NTc0Mzc1OS4zNy4wLjA."
-    (at 260.35 119.38 0)
+    (at 262.89 115.57 0)
     (effects (font (size 0.5 0.5)) (justify left bottom))
   )
@@
     (effects (font (size 1.27 1.27)) (justify right bottom))
   )
-  (global_label "M_TX" (shape input) (at 247.65 114.3 0) (fields_autoplaced)
+  (global_label "M_UART_TX" (shape input) (at 247.65 114.3 0) (fields_autoplaced)
     (effects (font (size 1.27 1.27)) (justify left))
-    (property "Intersheetrefs" "${INTERSHEET_REFS}" (at 255.2313 114.3 0)
+    (property "Intersheetrefs" "${INTERSHEET_REFS}" (at 260.8556 114.3 0)
       (effects (font (size 1.27 1.27)) (justify left) hide)
     )
@@
     )
   )
-  (global_label "M_RX" (shape output) (at 248.92 116.84 0) (fields_autoplaced)
+  (global_label "M_UART_RX" (shape output) (at 248.92 116.84 0) (fields_autoplaced)
     (effects (font (size 1.27 1.27)) (justify left))
-    (property "Intersheetrefs" "${INTERSHEET_REFS}" (at 256.8037 116.84 0)
+    (property "Intersheetrefs" "${INTERSHEET_REFS}" (at 262.428 116.84 0)
       (effects (font (size 1.27 1.27)) (justify left) hide)
     )

Commit message: more Zecong edits
Parts:
- added R? (x3): R_US, symbol Device:R_US
Connections:
- net +3V3: now also R?.1
- net GND: now also R?.2, R?.2
- net GPS_POWER: no longer Q4.3 (D)
- net IMU_POWER: now also Q4.3 (D), R?.2
- net at Q2.1 (B), R8.2: now also R?.1 (x2)
Other:
- note added: "Just incase everything goes terribly wrong"
- note added: "Mode 1 because we don't need it to be I2C master"
- note removed: "mode 1 because we don't need it to be I2C master"
- moved on the sheet: Q2, Q4, R7, R8
