File: boardlock/sensors.kicad_sch (KiCad schematic)
At the start: 34 parts, among them Q2 MMBT4401, Q4 BSS84PWH6327XTSA1, U1 LSM6DSO32, U3 SAM-M8Q

Commit message: buttons and stuff
Parts:
- removed TP15: GPS_POWER, symbol Connector:TestPoint
- removed TP16: IMU_POWER, symbol Connector:TestPoint
- removed TP4: GPS_EXTINT, symbol Connector:TestPoint
- removed TP9: IMU_INT2, symbol Connector:TestPoint
Changed lines of the file:
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@@
-    (stroke (width 0) (type default))
-  )
-  (wire (pts (xy 99.06 173.99) (xy 100.33 173.99))
     (stroke (width 0) (type default))
   )
@@
     (stroke (width 0) (type default))
   )
-  (wire (pts (xy 212.09 154.94) (xy 213.36 154.94))
-    (stroke (width 0) (type default))
-  )
   (wire (pts (xy 60.96 55.88) (xy 60.96 57.15))
     (stroke (width 0) (type default))
@@
     (stroke (width 0) (type default))
   )
-  (wire (pts (xy 99.06 177.8) (xy 100.33 177.8))
-    (stroke (width 0) (type default))
-  )
   (wire (pts (xy 88.9 110.49) (xy 88.9 123.19))
     (stroke (width 0) (type default))
@@
   )
   (wire (pts (xy 191.77 38.1) (xy 209.55 38.1))
-    (stroke (width 0) (type default))
-  )
-  (wire (pts (xy 212.09 158.75) (xy 213.36 158.75))
     (stroke (width 0) (type default))
   )
@@
     )
   )
-  (global_label "M_GPS_POWER" (shape input) (at 212.09 154.94 180) (fields_autoplaced)
-    (effects (font (size 1.27 1.27)) (justify right))
-    (property "Intersheetrefs" "${INTERSHEET_REFS}" (at 195.4978 154.94 0)
-      (effects (font (size 1.27 1.27)) (justify right) hide)
-    )
-  )
-  (global_label "M_IMU_POWER" (shape input) (at 99.06 173.99 180) (fields_autoplaced)
-    (effects (font (size 1.27 1.27)) (justify right))
-    (property "Intersheetrefs" "${INTERSHEET_REFS}" (at 82.8306 173.99 0)
-      (effects (font (size 1.27 1.27)) (justify right) hide)
-    )
-  )
-  (global_label "M_IMU_INT2" (shape input) (at 99.06 177.8 180) (fields_autoplaced)
-    (effects (font (size 1.27 1.27)) (justify right))
-    (property "Intersheetrefs" "${INTERSHEET_REFS}" (at 85.1891 177.8 0)
-      (effects (font (size 1.27 1.27)) (justify right) hide)
-    )
-  )
   (global_label "M_I2C_SDA" (shape bidirectional) (at 247.65 121.92 0) (fields_autoplaced)
     (effects (font (size 1.27 1.27)) (justify left))
@@
     )
   )
-  (global_label "M_GPS_EXTINT" (shape input) (at 212.09 158.75 180) (fields_autoplaced)
-    (effects (font (size 1.27 1.27)) (justify right))
-    (property "Intersheetrefs" "${INTERSHEET_REFS}" (at 195.7397 158.75 0)
-      (effects (font (size 1.27 1.27)) (justify right) hide)
-    )
-  )
   (global_label "M_UART_RX" (shape output) (at 248.92 116.84 0) (fields_autoplaced)
     (effects (font (size 1.27 1.27)) (justify left))
@@
     )
   )
-  (symbol (lib_id "Connector:TestPoint") (at 213.36 154.94 270) (unit 1)
-    (in_bom yes) (on_board yes) (dnp no)
-    (property "Reference" "TP15" (at 219.71 154.94 90)
-      (effects (font (size 1.27 1.27)))
-    )
-    (property "Value" "GPS_POWER" (at 229.87 154.94 90)
-      (effects (font (size 1.27 1.27)))
-    )
-    (property "Footprint" "" (at 213.36 160.02 0)
-      (effects (font (size 1.27 1.27)) hide)
-    )
-    (property "Datasheet" "~" (at 213.36 160.02 0)
-      (effects (font (size 1.27 1.27)) hide)
-    )
-    (pin "1")
-    (instances
-      (project "boardlock"
-        (path "/e1fc29ce-837e-4062-84d8-c7e423f9eab9/a4a6f965-a4d9-4da6-b64e-79eda0daabe5"
-          (reference "TP15") (unit 1)
-        )
-        (path "/e1fc29ce-837e-4062-84d8-c7e423f9eab9/ace912f2-c3e9-4bf3-99ba-49d1d353f0f6"
-          (reference "TP4") (unit 1)
-        )
-      )
-    )
-  )
   (symbol (lib_id "Connector:TestPoint") (at 199.39 119.38 90) (unit 1)
     (in_bom yes) (on_board yes) (dnp no)
@@
         (path "/e1fc29ce-837e-4062-84d8-c7e423f9eab9/a4a6f965-a4d9-4da6-b64e-79eda0daabe5"
           (reference "TP21") (unit 1)
-        )
-      )
-    )
-  )
-  (symbol (lib_id "Connector:TestPoint") (at 213.36 158.75 270) (unit 1)
-    (in_bom yes) (on_board yes) (dnp no)
-    (property "Reference" "TP4" (at 219.71 158.75 90)
-      (effects (font (size 1.27 1.27)))
-    )
-    (property "Value" "GPS_EXTINT" (at 229.87 158.75 90)
-      (effects (font (size 1.27 1.27)))
-    )
-    (property "Footprint" "" (at 213.36 163.83 0)
-      (effects (font (size 1.27 1.27)) hide)
-    )
-    (property "Datasheet" "~" (at 213.36 163.83 0)
-      (effects (font (size 1.27 1.27)) hide)
-    )
-    (pin "1")
-    (instances
-      (project "boardlock"
-        (path "/e1fc29ce-837e-4062-84d8-c7e423f9eab9/a4a6f965-a4d9-4da6-b64e-79eda0daabe5"
-          (reference "TP4") (unit 1)
-        )
-        (path "/e1fc29ce-837e-4062-84d8-c7e423f9eab9/ace912f2-c3e9-4bf3-99ba-49d1d353f0f6"
-          (reference "TP4") (unit 1)
         )
       )
@@
     )
   )
-  (symbol (lib_id "Connector:TestPoint") (at 100.33 173.99 270) (unit 1)
-    (in_bom yes) (on_board yes) (dnp no)
-    (property "Reference" "TP16" (at 106.68 173.99 90)
-      (effects (font (size 1.27 1.27)))
-    )
-    (property "Value" "IMU_POWER" (at 116.84 173.99 90)
-      (effects (font (size 1.27 1.27)))
-    )
-    (property "Footprint" "" (at 100.33 179.07 0)
-      (effects (font (size 1.27 1.27)) hide)
-    )
-    (property "Datasheet" "~" (at 100.33 179.07 0)
-      (effects (font (size 1.27 1.27)) hide)
-    )
-    (pin "1")
-    (instances
-      (project "boardlock"
-        (path "/e1fc29ce-837e-4062-84d8-c7e423f9eab9/a4a6f965-a4d9-4da6-b64e-79eda0daabe5"
-          (reference "TP16") (unit 1)
-        )
-        (path "/e1fc29ce-837e-4062-84d8-c7e423f9eab9/ace912f2-c3e9-4bf3-99ba-49d1d353f0f6"
-          (reference "TP4") (unit 1)
-        )
-      )
-    )
-  )
   (symbol (lib_id "power:+3V3") (at 191.77 34.29 0) (unit 1)
     (in_bom yes) (on_board yes) (dnp no) (fields_autoplaced)
@@
         )
       )
-    )
-  )
-  (symbol (lib_id "Connector:TestPoint") (at 100.33 177.8 270) (unit 1)
-    (in_bom yes) (on_board yes) (dnp no)
-    (property "Reference" "TP9" (at 106.68 177.8 90)
-      (effects (font (size 1.27 1.27)))
-    )
-    (property "Value" "IMU_INT2" (at 116.84 177.8 90)
-      (effects (font (size 1.27 1.27)))
-    )
-    (property "Footprint" "" (at 100.33 182.88 0)
-      (effects (font (size 1.27 1.27)) hide)
-    )
-    (property "Datasheet" "~" (at 100.33 182.88 0)
-      (effects (font (size 1.27 1.27)) hide)
-    )
-    (pin "1")
-    (instances
-      (project "boardlock"
-        (path "/e1fc29ce-837e-4062-84d8-c7e423f9eab9/a4a6f965-a4d9-4da6-b64e-79eda0daabe5"
-          (reference "TP9") (unit 1)
-        )
-        (path "/e1fc29ce-837e-4062-84d8-c7e423f9eab9/ace912f2-c3e9-4bf3-99ba-49d1d353f0f6"
-          (reference "TP4") (unit 1)
-        )
-      )

Commit message: lab updates
Parts:
- added R28: R_US, symbol Device:R_US
- added R9: 150k, symbol Device:R_US
- added R9: 200k, symbol Device:R_US
Connections:
- net +3V3: now also R28.1, R9.2
- net BACKUP: now also R9.1, R9.2
- net GND: now also R9.1
- net GPS_POWER: now also R28.2
Other:
- note added: "TEST THAT CS SHOULD BE HOOKED TO IMU_POWER"
- note added: "set values"
Changed lines of the file:
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@@
   (junction (at 69.85 135.89) (diameter 0) (color 0 0 0 0)
   )
+  (junction (at 242.57 59.69) (diameter 0) (color 0 0 0 0)
+  )
   (junction (at 274.32 59.69) (diameter 0) (color 0 0 0 0)
   )
@@
     (stroke (width 0) (type default))
   )
+  (wire (pts (xy 228.6 147.32) (xy 228.6 151.13))
+    (stroke (width 0) (type default))
+  )
   (wire (pts (xy 245.11 114.3) (xy 247.65 114.3))
     (stroke (width 0) (type default))
@@
     (stroke (width 0) (type default))
   )
+  (wire (pts (xy 228.6 161.29) (xy 237.49 161.29))
+    (stroke (width 0) (type default))
+  )
   (wire (pts (xy 60.96 64.77) (xy 60.96 66.04))
     (stroke (width 0) (type default))
   )
+  (wire (pts (xy 228.6 158.75) (xy 228.6 161.29))
+    (stroke (width 0) (type default))
+  )
   (wire (pts (xy 57.15 55.88) (xy 60.96 55.88))
     (stroke (width 0) (type default))
@@
     (stroke (width 0) (type default))
   )
+  (wire (pts (xy 242.57 59.69) (xy 245.11 59.69))
+    (stroke (width 0) (type default))
+  )
   (wire (pts (xy 73.66 38.1) (xy 73.66 35.56))
     (stroke (width 0) (type default))
@@
     (stroke (width 0) (type default))
   )
+  (wire (pts (xy 242.57 58.42) (xy 242.57 59.69))
+    (stroke (width 0) (type default))
+  )
   (wire (pts (xy 191.77 50.8) (xy 191.77 53.34))
     (stroke (width 0) (type default))
@@
   )
   (wire (pts (xy 199.39 121.92) (xy 200.66 121.92))
+    (stroke (width 0) (type default))
+  )
+  (wire (pts (xy 242.57 59.69) (xy 242.57 60.96))
     (stroke (width 0) (type default))
   )
@@
     (at 154.94 92.71 0)
     (effects (font (size 1.27 1.27)) (justify left bottom))
+  )
+  (text "set values\n" (at 243.84 62.23 0)
+    (effects (font (size 1.27 1.27) bold) (justify left bottom))
   )
   (text "ceramic" (at 64.77 121.92 0)
@@
     (effects (font (size 0.5 0.5)) (justify left bottom))
   )
+  (text "TEST THAT CS SHOULD BE HOOKED TO IMU_POWER\n" (at 33.02 156.21 0)
+    (effects (font (size 1.27 1.27) bold) (justify left bottom))
+  )
   (text "GPS Module" (at 191.77 91.44 0)
     (effects (font (size 1.27 1.27)) (justify left bottom))
@@
     (effects (font (size 5 5) (thickness 1) bold) (justify left bottom))
   )
+  (text "Just incase everything\ngoes terribly wrong" (at 240.03 153.67 0)
+    (effects (font (size 1.27 1.27)) (justify left bottom))
+  )
   (text "I2C Addr: 0x42\nchange by setting slaveAddr field \nof mode range: 0x07 < slaveAddr < 0x78. \nBit 0 must be 0\nSee 32.10.25.5 Port configuration for \nI2C (DDC) port of ReceiverDescrProtSpec"
     (at 157.48 146.05 0)
@@
     (effects (font (size 1.27 1.27)) (justify left bottom))
   )
-  (text "KEEP?\n" (at 245.11 46.99 0)
+  (text "KEEP?\n" (at 251.46 44.45 0)
     (effects (font (size 1.27 1.27) (thickness 0.254) bold) (justify left bottom))
   )
@@
     (effects (font (size 1.27 1.27)) (justify left bottom))
   )
+  (label "BACKUP" (at 245.11 59.69 0) (fields_autoplaced)
+    (effects (font (size 1.27 1.27)) (justify left bottom))
+  )
   (label "IMU_POWER" (at 71.12 146.05 180) (fields_autoplaced)
     (effects (font (size 1.27 1.27)) (justify right bottom))
@@
   (label "IMU_POWER" (at 62.23 106.68 180) (fields_autoplaced)
     (effects (font (size 1.27 1.27)) (justify right bottom))
+  )
+  (label "GPS_POWER" (at 237.49 161.29 0) (fields_autoplaced)
+    (effects (font (size 1.27 1.27)) (justify left bottom))
   )
   (label "GPS_POWER" (at 218.44 62.23 0) (fields_autoplaced)
@@
     )
   )
+  (symbol (lib_id "power:GND") (at 242.57 68.58 0) (unit 1)
+    (in_bom yes) (on_board yes) (dnp no) (fields_autoplaced)
+    (property "Reference" "#PWR01" (at 242.57 74.93 0)
+      (effects (font (size 1.27 1.27)) hide)
+    )
+    (property "Value" "GND" (at 242.57 72.7131 0)
+      (effects (font (size 1.27 1.27)))
+    )
+    (property "Footprint" "" (at 242.57 68.58 0)
+      (effects (font (size 1.27 1.27)) hide)
+    )
+    (property "Datasheet" "" (at 242.57 68.58 0)
+      (effects (font (size 1.27 1.27)) hide)
+    )
+    (pin "1")
+    (instances
+      (project "boardlock"
+        (path "/48f24f42-fd64-4860-9f12-ca34cf195758/17b4aebf-aea4-4bb2-a07c-86de8cf47820"
+          (reference "#PWR01") (unit 1)
+        )
+      )
+      (project "boardlock"
+        (path "/e1fc29ce-837e-4062-84d8-c7e423f9eab9/a4a6f965-a4d9-4da6-b64e-79eda0daabe5"
+          (reference "#PWR083") (unit 1)
+        )
+      )
+    )
+  )
   (symbol (lib_id "Connector:TestPoint") (at 199.39 119.38 90) (unit 1)
     (in_bom yes) (on_board yes) (dnp no)
@@
     )
   )
+  (symbol (lib_id "Device:R_US") (at 242.57 54.61 180) (unit 1)
+    (in_bom yes) (on_board yes) (dnp no)
+    (property "Reference" "R9" (at 240.03 54.61 90)
+      (effects (font (size 1.27 1.27)))
+    )
+    (property "Value" "150k" (at 245.11 54.61 90)
+      (effects (font (size 1.27 1.27)))
+    )
+    (property "Footprint" "" (at 241.554 54.356 90)
+      (effects (font (size 1.27 1.27)) hide)
+    )
+    (property "Datasheet" "~" (at 242.57 54.61 0)
+      (effects (font (size 1.27 1.27)) hide)
+    )
+    (pin "1")
+    (pin "2")
+    (instances
+      (project "boardlock"
+        (path "/48f24f42-fd64-4860-9f12-ca34cf195758/17b4aebf-aea4-4bb2-a07c-86de8cf47820"
+          (reference "R9") (unit 1)
+        )
+      )
+      (project "boardlock"
+        (path "/e1fc29ce-837e-4062-84d8-c7e423f9eab9/a4a6f965-a4d9-4da6-b64e-79eda0daabe5"
+          (reference "R26") (unit 1)
+        )
+      )
+    )
+  )
   (symbol (lib_id "Connector:TestPoint") (at 105.41 130.81 270) (unit 1)
     (in_bom yes) (on_board yes) (dnp no)
@@
         (path "/e1fc29ce-837e-4062-84d8-c7e423f9eab9/a4a6f965-a4d9-4da6-b64e-79eda0daabe5"
           (reference "TP21") (unit 1)
+        )
+      )
+    )
+  )
+  (symbol (lib_id "Device:R_US") (at 228.6 154.94 0) (unit 1)
+    (in_bom yes) (on_board yes) (dnp no) (fields_autoplaced)
+    (property "Reference" "R28" (at 231.14 153.67 0)
+      (effects (font (size 1.27 1.27)) (justify left))
+    )
+    (property "Value" "R_US" (at 231.14 156.21 0)
+      (effects (font (size 1.27 1.27)) (justify left))
+    )
+    (property "Footprint" "" (at 229.616 155.194 90)
+      (effects (font (size 1.27 1.27)) hide)
+    )
+    (property "Datasheet" "~" (at 228.6 154.94 0)
+      (effects (font (size 1.27 1.27)) hide)
+    )
+    (pin "1")
+    (pin "2")
+    (instances
+      (project "boardlock"
+        (path "/e1fc29ce-837e-4062-84d8-c7e423f9eab9/a4a6f965-a4d9-4da6-b64e-79eda0daabe5"
+          (reference "R28") (unit 1)
         )
       )
@@
         (path "/e1fc29ce-837e-4062-84d8-c7e423f9eab9/a4a6f965-a4d9-4da6-b64e-79eda0daabe5"
           (reference "C3") (unit 1)
+        )
+      )
+    )
+  )
+  (symbol (lib_id "Device:R_US") (at 242.57 64.77 180) (unit 1)
+    (in_bom yes) (on_board yes) (dnp no)
+    (property "Reference" "R9" (at 240.03 64.77 90)
+      (effects (font (size 1.27 1.27)))
+    )
+    (property "Value" "200k" (at 245.11 64.77 90)
+      (effects (font (size 1.27 1.27)))
+    )
+    (property "Footprint" "" (at 241.554 64.516 90)
+      (effects (font (size 1.27 1.27)) hide)
+    )
+    (property "Datasheet" "~" (at 242.57 64.77 0)
+      (effects (font (size 1.27 1.27)) hide)
+    )
+    (pin "1")
+    (pin "2")
+    (instances
+      (project "boardlock"
+        (path "/48f24f42-fd64-4860-9f12-ca34cf195758/17b4aebf-aea4-4bb2-a07c-86de8cf47820"
+          (reference "R9") (unit 1)
+        )
+      )
+      (project "boardlock"
+        (path "/e1fc29ce-837e-4062-84d8-c7e423f9eab9/a4a6f965-a4d9-4da6-b64e-79eda0daabe5"
+          (reference "R27") (unit 1)
         )
       )
@@
     )
   )
+  (symbol (lib_id "power:+3V3") (at 242.57 50.8 0) (unit 1)
+    (in_bom yes) (on_board yes) (dnp no) (fields_autoplaced)
+    (property "Reference" "#PWR09" (at 242.57 54.61 0)
+      (effects (font (size 1.27 1.27)) hide)
+    )
+    (property "Value" "+3V3" (at 242.57 46.6669 0)
+      (effects (font (size 1.27 1.27)))
+    )
+    (property "Footprint" "" (at 242.57 50.8 0)
+      (effects (font (size 1.27 1.27)) hide)
+    )
+    (property "Datasheet" "" (at 242.57 50.8 0)
+      (effects (font (size 1.27 1.27)) hide)
+    )
+    (pin "1")
+    (instances
+      (project "boardlock"
+        (path "/48f24f42-fd64-4860-9f12-ca34cf195758/17b4aebf-aea4-4bb2-a07c-86de8cf47820"
+          (reference "#PWR09") (unit 1)
+        )
+      )
+      (project "boardlock"
+        (path "/e1fc29ce-837e-4062-84d8-c7e423f9eab9/a4a6f965-a4d9-4da6-b64e-79eda0daabe5"
+          (reference "#PWR082") (unit 1)
+        )
+      )
+    )
+  )
   (symbol (lib_id "Device:R_US") (at 55.88 140.97 90) (unit 1)
     (in_bom yes) (on_board yes) (dnp no) (fields_autoplaced)
@@
         )
       )
+    )
+  )
+  (symbol (lib_id "power:+3V3") (at 228.6 147.32 0) (unit 1)
+    (in_bom yes) (on_board yes) (dnp no) (fields_autoplaced)
+    (property "Reference" "#PWR084" (at 228.6 151.13 0)
+      (effects (font (size 1.27 1.27)) hide)
+    )
+    (property "Value" "+3V3" (at 228.6 142.24 0)
+      (effects (font (size 1.27 1.27)))
+    )
+    (property "Footprint" "" (at 228.6 147.32 0)
+      (effects (font (size 1.27 1.27)) hide)
+    )
+    (property "Datasheet" "" (at 228.6 147.32 0)
+      (effects (font (size 1.27 1.27)) hide)
+    )
+    (pin "1")
+    (instances
+      (project "boardlock"
+        (path "/e1fc29ce-837e-4062-84d8-c7e423f9eab9/a4a6f965-a4d9-4da6-b64e-79eda0daabe5"
+          (reference "#PWR084") (unit 1)
+        )
+      )
