File: boardlock/boardlock.kicad_pcb (KiCad board)
At the start: 2 copper layers, 0 parts

Commit message: Nick PCB edits
Parts:
- added C1: 10uF, Capacitor_SMD:C_0805_2012Metric_Pad1.18x1.45mm_HandSolder, B.Cu at (74.5, 59.2)
- added C10: 22uF, Capacitor_SMD:C_0805_2012Metric_Pad1.18x1.45mm_HandSolder, F.Cu at (274.1, 339.9)
- added C11: 22uF, Capacitor_SMD:C_0805_2012Metric_Pad1.18x1.45mm_HandSolder, F.Cu at (274.1, 342.9)
- added C12: 22uF, Capacitor_SMD:C_0805_2012Metric_Pad1.18x1.45mm_HandSolder, F.Cu at (274.1, 345.9)
- added C13: 10uF, Capacitor_SMD:C_0805_2012Metric_Pad1.18x1.45mm_HandSolder, F.Cu at (461.6, 159.8)
- added C14: 0.1uF, Capacitor_SMD:C_0603_1608Metric_Pad1.08x0.95mm_HandSolder, F.Cu at (453.8, 158.2)
- added C15: 10uF, Capacitor_SMD:C_1206_3216Metric_Pad1.33x1.80mm_HandSolder, F.Cu at (150.1, 343.5)
- added C16: 10uF, Capacitor_SMD:C_0805_2012Metric_Pad1.18x1.45mm_HandSolder, F.Cu at (165.0, 338.6)
- added C17: 10uF, Capacitor_SMD:C_1206_3216Metric_Pad1.33x1.80mm_HandSolder, F.Cu at (158.7, 346.1)
- added C18: 1uF, Capacitor_SMD:C_0805_2012Metric_Pad1.18x1.45mm_HandSolder, B.Cu at (113.5, 92.2)
- added C19: 10uF, Capacitor_SMD:C_0805_2012Metric_Pad1.18x1.45mm_HandSolder, F.Cu at (95.8, 90.9)
- added C2: 0.1uF, Capacitor_SMD:C_0805_2012Metric_Pad1.18x1.45mm_HandSolder, B.Cu at (74.5, 61.4)
- added C20: 10uF, Capacitor_SMD:C_0805_2012Metric_Pad1.18x1.45mm_HandSolder, B.Cu at (109.5, 91.9)
- added C21: 0.47uF, Capacitor_SMD:C_0805_2012Metric_Pad1.18x1.45mm_HandSolder, F.Cu at (-112.8, 208.3)
- added C22: 1.0uF, Capacitor_SMD:C_0805_2012Metric_Pad1.18x1.45mm_HandSolder, F.Cu at (199.4, -79.1)
- added C23: 0.1uF, Capacitor_SMD:C_0805_2012Metric_Pad1.18x1.45mm_HandSolder, B.Cu at (76.2, 66.7)
- added C24: 0.1uF, Capacitor_SMD:C_0805_2012Metric_Pad1.18x1.45mm_HandSolder, B.Cu at (89.3, 49.0)
- added C25: 1uF, Capacitor_SMD:C_0805_2012Metric_Pad1.18x1.45mm_HandSolder, F.Cu at (-112.3, 210.8)
- added C26: 0.1uF, Capacitor_SMD:C_0805_2012Metric_Pad1.18x1.45mm_HandSolder, F.Cu at (294.6, -88.9)
- added C27: 0.1uF, Capacitor_SMD:C_0805_2012Metric_Pad1.18x1.45mm_HandSolder, F.Cu at (294.6, -85.9)
- added C28: 0.1uF, Capacitor_SMD:C_0805_2012Metric_Pad1.18x1.45mm_HandSolder, F.Cu at (396.0, -76.0)
- added C29: 10uF, Capacitor_SMD:C_0805_2012Metric_Pad1.18x1.45mm_HandSolder, F.Cu at (165.0, 341.6)
- added C3: 100nF, Capacitor_SMD:C_0805_2012Metric_Pad1.18x1.45mm_HandSolder, F.Cu at (90.4, -70.4)
- added C30: 10uF, Capacitor_SMD:C_0805_2012Metric_Pad1.18x1.45mm_HandSolder, F.Cu at (461.6, 162.8)
- added C31: 47n, Capacitor_SMD:C_0805_2012Metric_Pad1.18x1.45mm_HandSolder, F.Cu at (461.6, 165.8)
- added C32: 47n, Capacitor_SMD:C_0805_2012Metric_Pad1.18x1.45mm_HandSolder, F.Cu at (461.6, 168.8)
- added C33: 47n, Capacitor_SMD:C_0805_2012Metric_Pad1.18x1.45mm_HandSolder, F.Cu at (461.6, 171.8)
- added C34: 10uF, Capacitor_SMD:C_0805_2012Metric_Pad1.18x1.45mm_HandSolder, B.Cu at (74.7, 79.5)
- added C4: 100nF, Capacitor_SMD:C_0805_2012Metric_Pad1.18x1.45mm_HandSolder, F.Cu at (90.4, -67.4)
- added C5: 22uF, Capacitor_SMD:C_0805_2012Metric_Pad1.18x1.45mm_HandSolder, F.Cu at (274.1, 333.9)
- added C6: 22uF, Capacitor_SMD:C_0805_2012Metric_Pad1.18x1.45mm_HandSolder, F.Cu at (274.1, 336.9)
- added C7: 10uF, Capacitor_SMD:C_0603_1608Metric_Pad1.08x0.95mm_HandSolder, F.Cu at (279.4, 342.9)
- added C8: 100nF, Capacitor_SMD:C_0603_1608Metric_Pad1.08x0.95mm_HandSolder, F.Cu at (279.4, 345.4)
- added C9: 10uF, Capacitor_SMD:C_0603_1608Metric_Pad1.08x0.95mm_HandSolder, F.Cu at (279.4, 347.9)
- added D1: PMEG2005EH, Diode_SMD:D_SOD-123F, F.Cu at (163.9, 346.1)
- added D2: 1N5819HW1-7-F, Diode_SMD:D_SOD-123, B.Cu at (75.2, 74.7)
- added D3: LED, LED_SMD:LED_0805_2012Metric_Pad1.15x1.40mm_HandSolder, F.Cu at (-166.6, 71.1)
- added D4: CLVBA-FKA-CC1F1L1BB7R3R3D, LED_SMD:LED_Cree-PLCC4_3.2x2.8mm_CCW, F.Cu at (461.0, 19.1)
- added FB1: 4.7uH, Inductor_SMD:L_1210_3225Metric_Pad1.42x2.65mm_HandSolder, F.Cu at (454.0, 174.3)
- added FB2: 4.7uH, Inductor_SMD:L_1210_3225Metric_Pad1.42x2.65mm_HandSolder, F.Cu at (454.0, 178.5)
- added H1: MountingHole, MountingHole:MountingHole_2.2mm_M2, F.Cu at (-27.9, -65.7)
- added H2: MountingHole, MountingHole:MountingHole_2.2mm_M2, F.Cu at (-27.9, -55.6)
- added H3: MountingHole, MountingHole:MountingHole_2.2mm_M2, F.Cu at (-17.8, -65.7)
- added H4: MountingHole, MountingHole:MountingHole_2.2mm_M2, F.Cu at (-17.8, -55.6)
- added J1: Conn_01x02, Connector_JST:JST_PH_S2B-PH-K_1x02_P2.00mm_Horizontal, F.Cu at (-134.1, 142.2)
- added J2: Conn_01x02, Connector_JST:JST_PH_S2B-PH-K_1x02_P2.00mm_Horizontal, F.Cu at (73.1, 87.9)
- added J3: 5033981892, microSD 503398-1892:MOLEX_503398-1892, F.Cu at (377.1, 320.1)
- added J4: Conn_01x02, Connector_JST:JST_XA_B02B-XASK-1-A_1x02_P2.50mm_Vertical, F.Cu at (453.0, 165.8)
- added J5: Conn_01x02, Connector_JST:JST_XA_B02B-XASK-1-A_1x02_P2.50mm_Vertical, F.Cu at (439.4, 248.9)
- added J6: USB_C_Receptacle_USB2.0, Connector_USB:USB_C_Receptacle_GCT_USB4085, F.Cu at (67.3, 80.0)
- added L1: 1.5uH, DR74-1R5-R:DR74, F.Cu at (281.5, 337.2)
- added L2: 4.7uH, B82462G4472M000:IND_EPCOS_B82462G4_EPC, F.Cu at (157.7, 340.4)
- added Q1: BSS84PWH6327XTSA1, Package_TO_SOT_SMD:SOT-323_SC-70_Handsoldering, F.Cu at (87.6, -78.0)
- added Q2: MMBT4401, Package_TO_SOT_SMD:SOT-23-3, F.Cu at (95.4, -69.7)
- added Q3: MMBT4401, Package_TO_SOT_SMD:SOT-23-3, F.Cu at (204.3, -79.9)
- added Q4: BSS84PWH6327XTSA1, Package_TO_SOT_SMD:SOT-323_SC-70_Handsoldering, F.Cu at (210.8, -83.4)
- added Q5: MMBT4401, Package_TO_SOT_SMD:SOT-23-3, F.Cu at (471.3, 14.0)
- added Q6: MMBT4401, Package_TO_SOT_SMD:SOT-23-3, F.Cu at (471.3, 18.4)
- added Q7: MMBT4401, Package_TO_SOT_SMD:SOT-23-3, F.Cu at (471.3, 22.9)
- added Q8: BSS84PWH6327XTSA1, Package_TO_SOT_SMD:SOT-323_SC-70_Handsoldering, F.Cu at (444.2, 256.2)
- added Q9: MMBT4401, Package_TO_SOT_SMD:SOT-23-3, F.Cu at (449.4, 245.4)
- added R1: 470, Resistor_SMD:R_0805_2012Metric_Pad1.20x1.40mm_HandSolder, F.Cu at (201.0, -96.9)
- added R10: 150k, Resistor_SMD:R_0805_2012Metric_Pad1.20x1.40mm_HandSolder, F.Cu at (269.3, 336.8)
- added R11: 100k, Resistor_SMD:R_0805_2012Metric_Pad1.20x1.40mm_HandSolder, F.Cu at (269.3, 339.7)
- added R12: 5.1k, Resistor_SMD:R_0805_2012Metric_Pad1.20x1.40mm_HandSolder, B.Cu at (68.1, 83.6)
- added R13: 5.1k, Resistor_SMD:R_0805_2012Metric_Pad1.20x1.40mm_HandSolder, B.Cu at (74.7, 77.2)
- added R14: 10k, Resistor_SMD:R_0805_2012Metric_Pad1.20x1.40mm_HandSolder, F.Cu at (269.3, 342.7)
- added R15: 470, Resistor_SMD:R_0805_2012Metric_Pad1.20x1.40mm_HandSolder, F.Cu at (205.7, -88.1)
- added R16: R_US, Resistor_SMD:R_0805_2012Metric_Pad1.20x1.40mm_HandSolder, F.Cu at (92.1, -73.4)
- added R17: 5.1k, Resistor_SMD:R_0805_2012Metric_Pad1.20x1.40mm_HandSolder, F.Cu at (66.2, 35.3)
- added R18: 10k, Resistor_SMD:R_0805_2012Metric_Pad1.20x1.40mm_HandSolder, F.Cu at (108.3, 67.5)
- added R19: 5.1k, Resistor_SMD:R_0805_2012Metric_Pad1.20x1.40mm_HandSolder, F.Cu at (69.9, 34.0)
- added R2: R_US, Resistor_SMD:R_0805_2012Metric_Pad1.20x1.40mm_HandSolder, F.Cu at (77.7, -73.8)
- added R20: 1k, Resistor_SMD:R_0805_2012Metric_Pad1.20x1.40mm_HandSolder, F.Cu at (299.7, -88.9)
- added R21: 1k, Resistor_SMD:R_0805_2012Metric_Pad1.20x1.40mm_HandSolder, F.Cu at (299.7, -86.0)
- added R22: 1k, Resistor_SMD:R_0805_2012Metric_Pad1.20x1.40mm_HandSolder, F.Cu at (400.3, -73.7)
- added R23: 10k, Resistor_SMD:R_0805_2012Metric_Pad1.20x1.40mm_HandSolder, F.Cu at (101.3, 67.5)
- added R24: R_US, Resistor_SMD:R_0805_2012Metric_Pad1.20x1.40mm_HandSolder, F.Cu at (84.3, -70.6)
- added R25: R_US, Resistor_SMD:R_0805_2012Metric_Pad1.20x1.40mm_HandSolder, F.Cu at (210.5, -94.0)
- added R26: 0, Resistor_SMD:R_0805_2012Metric_Pad1.20x1.40mm_HandSolder, F.Cu at (103.4, 84.8)
- added R27: 0, Resistor_SMD:R_0805_2012Metric_Pad1.20x1.40mm_HandSolder, F.Cu at (98.0, 90.9)
- added R28: R_US, Resistor_SMD:R_0805_2012Metric_Pad1.20x1.40mm_HandSolder, F.Cu at (210.5, -91.0)
- added R29: R_US, Resistor_SMD:R_0805_2012Metric_Pad1.20x1.40mm_HandSolder, F.Cu at (-166.6, 73.7)
- added R3: R_US, Resistor_SMD:R_0805_2012Metric_Pad1.20x1.40mm_HandSolder, F.Cu at (77.7, -70.8)
- added R30: R_US, Resistor_SMD:R_0805_2012Metric_Pad1.20x1.40mm_HandSolder, F.Cu at (455.7, 12.5)
- added R31: R_US, Resistor_SMD:R_0805_2012Metric_Pad1.20x1.40mm_HandSolder, F.Cu at (455.7, 15.5)
- added R32: R_US, Resistor_SMD:R_0805_2012Metric_Pad1.20x1.40mm_HandSolder, F.Cu at (455.7, 18.4)
- added R33: R_US, Resistor_SMD:R_0805_2012Metric_Pad1.20x1.40mm_HandSolder, F.Cu at (455.7, 21.4)
- added R34: R_US, Resistor_SMD:R_0805_2012Metric_Pad1.20x1.40mm_HandSolder, F.Cu at (455.7, 24.3)
- added R35: R_US, Resistor_SMD:R_0805_2012Metric_Pad1.20x1.40mm_HandSolder, F.Cu at (466.4, 15.1)
- added R36: R_US, Resistor_SMD:R_0805_2012Metric_Pad1.20x1.40mm_HandSolder, F.Cu at (466.4, 18.0)
- added R37: R_US, Resistor_SMD:R_0805_2012Metric_Pad1.20x1.40mm_HandSolder, F.Cu at (466.4, 20.9)
- added R38: R_US, Resistor_SMD:R_0805_2012Metric_Pad1.20x1.40mm_HandSolder, F.Cu at (86.4, -72.9)
- added R39: R_US, Resistor_SMD:R_0805_2012Metric_Pad1.20x1.40mm_HandSolder, F.Cu at (466.4, 23.9)
- added R4: R_US, Resistor_SMD:R_0805_2012Metric_Pad1.20x1.40mm_HandSolder, F.Cu at (77.7, -67.9)
- added R40: 1.2k, Resistor_SMD:R_0805_2012Metric_Pad1.20x1.40mm_HandSolder, F.Cu at (92.5, 90.7)
- added R41: 5.1k, Resistor_SMD:R_0805_2012Metric_Pad1.20x1.40mm_HandSolder, F.Cu at (99.3, 84.8)
- added R42: 5.1k, Resistor_SMD:R_0805_2012Metric_Pad1.20x1.40mm_HandSolder, F.Cu at (100.3, 90.9)
- added R43: R_US, Resistor_SMD:R_0805_2012Metric_Pad1.20x1.40mm_HandSolder, F.Cu at (90.2, 90.7)
- added R44: 10k, Resistor_SMD:R_0805_2012Metric_Pad1.20x1.40mm_HandSolder, F.Cu at (90.2, 85.1)
- added R45: 47k, Resistor_SMD:R_0805_2012Metric_Pad1.20x1.40mm_HandSolder, F.Cu at (95.2, 81.8)
- added R46: 100k, Resistor_SMD:R_0805_2012Metric_Pad1.20x1.40mm_HandSolder, F.Cu at (90.2, 87.1)
- added R47: 1.2k, Resistor_SMD:R_0805_2012Metric_Pad1.20x1.40mm_HandSolder, F.Cu at (98.6, 82.5)
- added R48: 1.2k, Resistor_SMD:R_0805_2012Metric_Pad1.20x1.40mm_HandSolder, F.Cu at (93.0, 81.8)
- added R49: 10k, Resistor_SMD:R_0805_2012Metric_Pad1.20x1.40mm_HandSolder, F.Cu at (-112.8, 205.7)
- added R5: R_US, Resistor_SMD:R_0805_2012Metric_Pad1.20x1.40mm_HandSolder, F.Cu at (201.0, -85.1)
- added R50: 10m, Resistor_SMD:R_2512_6332Metric_Pad1.40x3.35mm_HandSolder, F.Cu at (-119.4, 210.8)
- added R51: 560k, Resistor_SMD:R_0805_2012Metric_Pad1.20x1.40mm_HandSolder, F.Cu at (269.3, 345.6)
- added R52: 330k, Resistor_SMD:R_0805_2012Metric_Pad1.20x1.40mm_HandSolder, F.Cu at (269.3, 348.6)
- added R53: 330k, Resistor_SMD:R_0805_2012Metric_Pad1.20x1.40mm_HandSolder, F.Cu at (269.3, 351.5)
- added R54: 1.05M, Resistor_SMD:R_0805_2012Metric_Pad1.20x1.40mm_HandSolder, F.Cu at (150.1, 338.1)
- added R55: 120k, Resistor_SMD:R_0805_2012Metric_Pad1.20x1.40mm_HandSolder, F.Cu at (150.1, 341.0)
- added R56: 100k, Resistor_SMD:R_0805_2012Metric_Pad1.20x1.40mm_HandSolder, F.Cu at (446.4, 167.9)
- added R57: 100k, Resistor_SMD:R_0805_2012Metric_Pad1.20x1.40mm_HandSolder, F.Cu at (446.4, 170.9)
- added R58: ?, Resistor_SMD:R_0805_2012Metric_Pad1.20x1.40mm_HandSolder, F.Cu at (446.4, 173.8)
- added R59: R_US, Resistor_SMD:R_0805_2012Metric_Pad1.20x1.40mm_HandSolder, F.Cu at (449.5, 250.1)
- added R6: R_US, Resistor_SMD:R_0805_2012Metric_Pad1.20x1.40mm_HandSolder, F.Cu at (205.7, -96.9)
- added R60: R_US, Resistor_SMD:R_0805_2012Metric_Pad1.20x1.40mm_HandSolder, F.Cu at (449.5, 253.1)
- added R61: R_US, Resistor_SMD:R_0805_2012Metric_Pad1.20x1.40mm_HandSolder, F.Cu at (449.5, 256.0)
- added R7: 22, Resistor_SMD:R_0805_2012Metric_Pad1.20x1.40mm_HandSolder, F.Cu at (205.7, -94.0)
- added R8: 22, Resistor_SMD:R_0805_2012Metric_Pad1.20x1.40mm_HandSolder, F.Cu at (205.7, -91.0)
- added R9: 470k, Resistor_SMD:R_0805_2012Metric_Pad1.20x1.40mm_HandSolder, F.Cu at (269.3, 333.8)
- added SW1: SW_Push, Button_Switch_SMD:SW_Push_1P1T_NO_Vertical_Wuerth_434133025816, F.Cu at (101.3, 70.9)
- added SW2: SW_Push, Button_Switch_SMD:SW_Push_1P1T_NO_Vertical_Wuerth_434133025816, F.Cu at (108.2, 70.9)
- added SW3: SW_Push, TL3300DF160Q:SW_TL3300DF160Q, F.Cu at (317.5, -76.2)
- added SW4: SW_Push, Button_Switch_SMD:SW_Push_1P1T_NO_Vertical_Wuerth_434133025816, F.Cu at (401.8, -77.7)
- added SW5: SW_Push, TL3300DF160Q:SW_TL3300DF160Q, F.Cu at (297.8, -76.2)
- added TP1: TIMEPULSE, TestPoint:TestPoint_Pad_D1.0mm, F.Cu at (180.3, -78.3)
- added TP10: TestPoint, TestPoint:TestPoint_Pad_D1.0mm, F.Cu at (-101.6, 4.58)
- added TP11: TestPoint, TestPoint:TestPoint_Pad_D1.0mm, F.Cu at (-101.6, 7.63)
- added TP12: TestPoint, TestPoint:TestPoint_Pad_D1.0mm, F.Cu at (-98.5, -13.7)
- added TP13: TestPoint, TestPoint:TestPoint_Pad_D1.0mm, F.Cu at (-98.5, -10.7)
- added TP14: TestPoint, TestPoint:TestPoint_Pad_D1.0mm, F.Cu at (-98.5, -7.62)
- added TP15: TestPoint, TestPoint:TestPoint_Pad_D1.0mm, F.Cu at (-98.5, -4.57)
- added TP16: TestPoint, TestPoint:TestPoint_Pad_D1.0mm, F.Cu at (-98.5, -1.52)
- added TP17: TestPoint, TestPoint:TestPoint_Pad_D1.0mm, F.Cu at (-98.5, 1.53)
- added TP18: TestPoint, TestPoint:TestPoint_Pad_D1.0mm, F.Cu at (-98.5, 4.58)
- added TP19: TestPoint, TestPoint:TestPoint_Pad_D1.0mm, F.Cu at (-98.5, 7.63)
- added TP2: GPS_RESET_N, TestPoint:TestPoint_Pad_D1.0mm, F.Cu at (180.3, -75.3)
- added TP20: TestPoint, TestPoint:TestPoint_Pad_D1.0mm, F.Cu at (-95.5, -13.7)
- added TP21: IMU_INT1, TestPoint:TestPoint_Pad_D1.0mm, F.Cu at (76.2, -78.0)
- added TP22: TestPoint, TestPoint:TestPoint_Pad_D1.0mm, F.Cu at (-95.5, -10.7)
- added TP23: TestPoint, TestPoint:TestPoint_Pad_D1.0mm, F.Cu at (-95.5, -7.62)
- added TP24: TestPoint, TestPoint:TestPoint_Pad_D1.0mm, F.Cu at (-95.5, -4.57)
- added TP25: TestPoint, TestPoint:TestPoint_Pad_D1.0mm, F.Cu at (-95.5, -1.52)
- added TP26: TestPoint, TestPoint:TestPoint_Pad_D1.0mm, F.Cu at (-95.5, 1.53)
- added TP27: TestPoint, TestPoint:TestPoint_Pad_D1.0mm, F.Cu at (-95.5, 4.58)
- added TP28: TestPoint, TestPoint:TestPoint_Pad_D1.0mm, F.Cu at (-95.5, 7.63)
- added TP29: TestPoint, TestPoint:TestPoint_Pad_D1.0mm, F.Cu at (-92.5, -13.7)
- added TP3: GPS_SAFE_N, TestPoint:TestPoint_Pad_D1.0mm, F.Cu at (180.3, -72.2)
- added TP30: TestPoint, TestPoint:TestPoint_Pad_D1.0mm, F.Cu at (-92.5, -10.7)
- added TP31: TestPoint, TestPoint:TestPoint_Pad_D1.0mm, F.Cu at (-92.5, -7.62)
- added TP32: TestPoint, TestPoint:TestPoint_Pad_D1.0mm, F.Cu at (-92.5, -4.57)
- added TP33: TestPoint, TestPoint:TestPoint_Pad_D1.0mm, F.Cu at (-92.5, -1.52)
- added TP34: TestPoint, TestPoint:TestPoint_Pad_D1.0mm, F.Cu at (-92.5, 1.53)
- added TP35: TestPoint, TestPoint:TestPoint_Pad_D1.0mm, F.Cu at (-92.5, 4.58)
- added TP36: TestPoint, TestPoint:TestPoint_Pad_D1.0mm, F.Cu at (-92.5, 7.63)
- added TP37: TestPoint, TestPoint:TestPoint_Pad_D1.0mm, F.Cu at (-89.4, -13.7)
- added TP38: TestPoint, TestPoint:TestPoint_Pad_D1.0mm, F.Cu at (-89.4, -10.7)
- added TP39: TestPoint, TestPoint:TestPoint_Pad_D1.0mm, F.Cu at (-89.4, -7.62)
- added TP4: TestPoint, TestPoint:TestPoint_Pad_D1.0mm, F.Cu at (-101.6, -13.7)
- added TP40: TestPoint, TestPoint:TestPoint_Pad_D1.0mm, F.Cu at (-89.4, 1.52)
- added TP41: TestPoint, TestPoint:TestPoint_Pad_D1.0mm, F.Cu at (-89.4, -4.57)
- added TP42: TestPoint, TestPoint:TestPoint_Pad_D1.0mm, F.Cu at (-89.4, -1.52)
- added TP43: TestPoint, TestPoint:TestPoint_Pad_D1.0mm, F.Cu at (-89.4, 4.57)
- added TP5: TestPoint, TestPoint:TestPoint_Pad_D1.0mm, F.Cu at (-101.6, -10.7)
- added TP6: TestPoint, TestPoint:TestPoint_Pad_D1.0mm, F.Cu at (-101.6, -7.62)
- added TP7: TestPoint, TestPoint:TestPoint_Pad_D1.0mm, F.Cu at (-101.6, -4.57)
- added TP8: TestPoint, TestPoint:TestPoint_Pad_D1.0mm, F.Cu at (-101.6, -1.52)
- added TP9: TestPoint, TestPoint:TestPoint_Pad_D1.0mm, F.Cu at (-101.6, 1.53)
- added U10: ESP32-S3-WROOM-1, espressif-kicad:ESP32-S3-WROOM-1, F.Cu at (81.9, 54.8)
- added U2: LSM6DSO32, Package_LGA:LGA-14_3x2.5mm_P0.5mm_LayoutBorder3x4y, F.Cu at (80.8, -77.1)
- added U3: SAM-M8Q, RF_GPS:ublox_SAM-M8Q, F.Cu at (186.9, -90.2)
- added U4: BQ24075RGT, Package_DFN_QFN:VQFN-16-1EP_3x3mm_P0.5mm_EP1.6x1.6mm, F.Cu at (94.8, 86.1)
- added U5: BQ27441DRZR-G1A, Package_SON:Texas_S-PDSO-N12, F.Cu at (-119.9, 205.3)
- added U6: TPS630701RNMR, TPS630701RNMR:TPS630701RNMR, F.Cu at (285.6, 345.6)
- added U7: MAX98357AETE+T, MAX98357AETE+T:QFN50P300X300X80-17N, F.Cu at (445.6, 161.8)
- added U8: MCP1661, Package_TO_SOT_SMD:SOT-23-5, F.Cu at (151.5, 347.0)
- added U9: TPD2E2U06, Package_TO_SOT_SMD:SOT-553, B.Cu at (71.1, 75.9)
Routing:
- net M_BOOT: track 0.00 -> 48.8 mm, vias 0 -> 2
- net M_RST_N: track 0.00 -> 36.7 mm, vias 0 -> 2
- net M_BUTTON_EXT1: track 0.00 -> 21.5 mm, vias 0 -> 1
- net M_BUTTON_EXT2: track 0.00 -> 20.0 mm, vias 0 -> 1
- net Net-(U10-U0TXD/GPIO43/CLK_OUT1): track 0.00 -> 18.5 mm, vias 0 -> 1
- net GND: track 0.00 -> 18.1 mm
- net Net-(U10-U0RXD/GPIO44/CLK_OUT2): track 0.00 -> 17.1 mm, vias 0 -> 1
- net M_RGB_B: track 0.00 -> 15.6 mm, vias 0 -> 1
- net M_RGB_G: track 0.00 -> 14.1 mm, vias 0 -> 1
- net M_RGB_R: track 0.00 -> 12.6 mm, vias 0 -> 1
- net Net-(U10-MTCK/GPIO39/CLK_OUT3/SUBSPICS1): track 0.00 -> 11.1 mm, vias 0 -> 1
- net M_BUTTON_INT: track 0.00 -> 9.65 mm, vias 0 -> 1
- net M_HEARTBEAT: track 0.00 -> 8.17 mm, vias 0 -> 1
- net /ui/V_USB: track 0.00 -> 7.72 mm, vias 0 -> 1
- net Net-(U10-SPIIO7/GPIO36/FSPICLK/SUBSPICLK): track 0.00 -> 6.69 mm, vias 0 -> 1
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Other:
- board outline added: 127 x 76.2 mm
- board text added: "12V Boost Converter"
- board text added: "3V3 Bust-Boost"
- board text added: "Audio Amplifier"
- board text added: "Babysitter Input"
- board text added: "Battery Charging"
- board text added: "Battery Gauge"
- board text added: "Buzzer Power Circuit"
- board text added: "External UI Buttons"
- board text added: "GPS"
- board text added: "Heart"
- board text added: "IMU"
- board text added: "LiPo Battery Connector"
- board text added: "MICRO"
- board text added: "MicroSD Slot"
- board text added: "Mount Holes"
- board text added: "NOT DON EYET"
- board text added: "Non-UI Buttons"
- board text added: "RGB"
- board text added: "Testpoints"
- board text added: "USB-C Connector"
- board text added: "User Data Reset Button"

Commit message: SOmething
Parts:
- moved C18 18.1 mm to (95.5, 91.1), turned to -90 degrees
- moved R26 13.6 mm to (90.1, 81.9), turned to -90 degrees
- moved R43 13.5 mm to (100.4, 81.9), turned to 90 degrees
- moved R42 12.1 mm to (92.3, 81.9), turned to -90 degrees
- moved R12 11.0 mm to (74.7, 74.8), turned to 90 degrees
- moved R44 10.5 mm to (100.4, 87.5), turned to 0 degrees
- moved R40 10.4 mm to (98.1, 81.9), turned to -90 degrees
- moved C20 10.4 mm to (100.6, 86.5), turned to 0 degrees
- moved R46 10.4 mm to (100.4, 85.5), turned to 0 degrees
- moved R48 10.2 mm to (97.6, 90.8), turned to -90 degrees
- moved R47 9.93 mm to (92.0, 90.0), turned to 180 degrees
- moved R27 9.67 mm to (94.6, 81.9), turned to -90 degrees
- moved R45 9.02 mm to (95.3, 90.8), turned to -90 degrees
- moved R41 8.57 mm to (90.8, 85.8), turned to 0 degrees
- moved J6 6.79 mm to (71.6, 74.8), turned to -90 degrees
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Routing:
- net GND: track 18.1 -> 37.6 mm, vias 0 -> 1
- net M_BATT_CHARGE_N_CHG: track 0.00 -> 6.16 mm
- net Net-(J6-CC2): track 5.86 -> 11.7 mm, vias 1 -> 2
- net BATT_CHARGE_EN2: track 0.00 -> 4.88 mm
- net BATT_CHARGE_VOUT: track 0.50 -> 4.03 mm
- net Net-(U4-ILIM): track 0.00 -> 3.33 mm
- net Net-(J6-CC1): track 6.46 -> 3.38 mm
- net +BATT: track 0.00 -> 2.95 mm, vias 0 -> 1
- net /ui/V_USB: track 7.72 -> 10.5 mm, vias 1 -> 0
- net M_BATT_CHARGE_N_PGOOD: track 2.29 -> 4.84 mm
- net Net-(U4-~{CE}): track 0.00 -> 2.34 mm
- net Net-(U4-ISET): track 0.00 -> 2.33 mm
- net TS_RESISTOR: track 0.00 -> 2.33 mm
- net Net-(U4-TMR): track 0.00 -> 1.94 mm
- net VBUS: track 5.29 -> 5.95 mm, vias 0 -> 1
Other:
- board text added: "3V3 Buck-Boost"
- board text added: "NOT DONE YET"
- board text removed: "3V3 Bust-Boost"
- board text removed: "NOT DON EYET"

Commit message: commit
Parts:
- moved U10 25.3 mm to (56.8, 57.8)
Routing:
- net M_RST_N: track 36.7 -> 10.3 mm, vias 2 -> 0
- net M_BOOT: track 48.8 -> 26.4 mm, vias 2 -> 0
- net M_BUTTON_EXT1: track 21.5 -> 0.00 mm, vias 1 -> 0
- net M_BUTTON_EXT2: track 20.0 -> 0.00 mm, vias 1 -> 0
- net Net-(U10-U0TXD/GPIO43/CLK_OUT1): track 18.5 -> 0.00 mm, vias 1 -> 0
- net Net-(U10-U0RXD/GPIO44/CLK_OUT2): track 17.1 -> 0.00 mm, vias 1 -> 0
- net M_RGB_B: track 15.6 -> 0.00 mm, vias 1 -> 0
- net M_RGB_G: track 14.1 -> 0.00 mm, vias 1 -> 0
- net M_RGB_R: track 12.6 -> 0.00 mm, vias 1 -> 0
- net Net-(U10-MTCK/GPIO39/CLK_OUT3/SUBSPICS1): track 11.1 -> 0.00 mm, vias 1 -> 0
- net M_BUTTON_INT: track 9.65 -> 0.00 mm, vias 1 -> 0
- net M_HEARTBEAT: track 8.17 -> 0.00 mm, vias 1 -> 0
- net Net-(U10-SPIIO7/GPIO36/FSPICLK/SUBSPICLK): track 6.69 -> 0.00 mm, vias 1 -> 0
- net M_IMU_INT2: track 5.11 -> 0.00 mm, vias 1 -> 0
Changed lines of the file:
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@@
   )
   (footprint "espressif-kicad:ESP32-S3-WROOM-1" (layer "F.Cu")
-    (at 81.92 54.75 90)
+    (at 56.774 57.772 90)
     (descr "ESP32-S3-WROOM-1 is a powerful, generic Wi-Fi + Bluetooth LE MCU modules that have Dual core CPU , a rich set of peripherals, provides acceleration for neural network computing and signal processing workloads. They are an ideal choice for a wide variety of application scenarios related to AI + Internet of Things (AIoT), such as wake word detection and speech commands recognition , face detection and recognition, smart home, smart appliance, smart control panel, smart speaker etc.")
     (tags "esp32-s3")
@@
       (polygon
         (pts
-          (xy 72.12 45.75)
-          (xy 72.12 63.75)
-          (xy 66.17 63.75)
-          (xy 66.17 45.75)
+          (xy 46.974 48.772)
+          (xy 46.974 66.772)
+          (xy 41.024 66.772)
+          (xy 41.024 48.772)
         )
       )
@@
   (segment (start 76.2 65.6) (end 76.2 63.5) (width 0.25) (layer "F.Cu") (net 11))
   (segment (start 103.4 68.6) (end 103.4 69.8) (width 0.254) (layer "F.Cu") (net 11))
-  (via (at 76.2 65.6) (size 0.8) (drill 0.4) (layers "F.Cu" "B.Cu") (net 11))
-  (via (at 102.3 66.2) (size 0.8) (drill 0.4) (layers "F.Cu" "B.Cu") (net 11))
-  (segment (start 76.2 65.6625) (end 76.2 65.6) (width 0.25) (layer "B.Cu") (net 11))
-  (segment (start 76.7375 66.2) (end 76.2 65.6625) (width 0.254) (layer "B.Cu") (net 11))
-  (segment (start 102.3 66.2) (end 76.7375 66.2) (width 0.254) (layer "B.Cu") (net 11))
-  (segment (start 89.3 48) (end 90.17 47.13) (width 0.254) (layer "F.Cu") (net 12))
-  (segment (start 90.17 47.13) (end 90.17 46) (width 0.254) (layer "F.Cu") (net 12))
   (segment (start 110.275 69.825) (end 106.15 69.825) (width 0.254) (layer "F.Cu") (net 12))
   (segment (start 110.275 68.475) (end 110.275 69.825) (width 0.254) (layer "F.Cu") (net 12))
   (segment (start 109.3 67.5) (end 110.275 68.475) (width 0.254) (layer "F.Cu") (net 12))
   (segment (start 109.3 48) (end 109.3 67.5) (width 0.254) (layer "F.Cu") (net 12))
-  (via (at 109.3 48) (size 0.8) (drill 0.4) (layers "F.Cu" "B.Cu") (net 12))
-  (via (at 89.3 48) (size 0.8) (drill 0.4) (layers "F.Cu" "B.Cu") (net 12))
-  (segment (start 89.3 47.9625) (end 89.3 48) (width 0.254) (layer "B.Cu") (net 12))
-  (segment (start 89.3 48) (end 109.3 48) (width 0.254) (layer "B.Cu") (net 12))
-  (segment (start 74.93 46) (end 74.93 44.45) (width 0.254) (layer "F.Cu") (net 14))
-  (via (at 74.93 44.45) (size 0.8) (drill 0.4) (layers "F.Cu" "B.Cu") (net 14))
-  (segment (start 80.772 38.608) (end 92.456 38.608) (width 0.254) (layer "B.Cu") (net 14))
-  (segment (start 74.93 44.45) (end 80.772 38.608) (width 0.254) (layer "B.Cu") (net 14))
-  (segment (start 76.2 46) (end 76.2 44.45) (width 0.254) (layer "F.Cu") (net 15))
-  (via (at 76.2 44.45) (size 0.8) (drill 0.4) (layers "F.Cu" "B.Cu") (net 15))
-  (segment (start 81.534 39.116) (end 92.456 39.116) (width 0.254) (layer "B.Cu") (net 15))
-  (segment (start 76.2 44.45) (end 81.534 39.116) (width 0.254) (layer "B.Cu") (net 15))
-  (segment (start 85.09 46) (end 85.09 44.45) (width 0.254) (layer "F.Cu") (net 16))
-  (via (at 85.09 44.45) (size 0.8) (drill 0.4) (layers "F.Cu" "B.Cu") (net 16))
-  (segment (start 85.09 44.45) (end 86.868 42.672) (width 0.254) (layer "B.Cu") (net 16))
-  (segment (start 86.868 42.672) (end 92.456 42.672) (width 0.254) (layer "B.Cu") (net 16))
   (segment (start 77.677 79.827) (end 71.723 79.827) (width 0.254) (layer "B.Cu") (net 20))
   (segment (start 70.275 79.925) (end 71.625 79.925) (width 0.254) (layer "B.Cu") (net 20))
@@
   (segment (start 71.8 83.4) (end 74.3 80.9) (width 0.254) (layer "B.Cu") (net 38))
   (segment (start 69.1 83.4) (end 71.8 83.4) (width 0.254) (layer "B.Cu") (net 38))
-  (segment (start 86.36 46) (end 86.36 44.45) (width 0.254) (layer "F.Cu") (net 72))
-  (via (at 86.36 44.45) (size 0.8) (drill 0.4) (layers "F.Cu" "B.Cu") (net 72))
-  (segment (start 87.63 43.18) (end 92.456 43.18) (width 0.254) (layer "B.Cu") (net 72))
-  (segment (start 86.36 44.45) (end 87.63 43.18) (width 0.254) (layer "B.Cu") (net 72))
-  (segment (start 82.55 46) (end 82.55 44.45) (width 0.254) (layer "F.Cu") (net 73))
-  (via (at 82.55 44.45) (size 0.8) (drill 0.4) (layers "F.Cu" "B.Cu") (net 73))
-  (segment (start 85.344 41.656) (end 92.456 41.656) (width 0.254) (layer "B.Cu") (net 73))
-  (segment (start 82.55 44.45) (end 85.344 41.656) (width 0.254) (layer "B.Cu") (net 73))
-  (segment (start 81.28 46) (end 81.28 44.45) (width 0.254) (layer "F.Cu") (net 74))
-  (via (at 81.28 44.45) (size 0.8) (drill 0.4) (layers "F.Cu" "B.Cu") (net 74))
-  (segment (start 84.582 41.148) (end 92.456 41.148) (width 0.254) (layer "B.Cu") (net 74))
-  (segment (start 81.28 44.45) (end 84.582 41.148) (width 0.254) (layer "B.Cu") (net 74))
-  (segment (start 80.01 46) (end 80.01 44.45) (width 0.254) (layer "F.Cu") (net 75))
-  (via (at 80.01 44.45) (size 0.8) (drill 0.4) (layers "F.Cu" "B.Cu") (net 75))
-  (segment (start 80.01 44.45) (end 83.82 40.64) (width 0.254) (layer "B.Cu") (net 75))
-  (segment (start 83.82 40.64) (end 92.456 40.64) (width 0.254) (layer "B.Cu") (net 75))
   (segment (start 96.0215 84.580164) (end 97.679664 82.922) (width 0.254) (layer "F.Cu") (net 76))
   (segment (start 96.0215 85.0685) (end 96.0215 84.580164) (width 0.254) (layer "F.Cu") (net 76))
@@
   (segment (start 96.5215 87.9435) (end 96.5215 88.6975) (width 0.254) (layer "F.Cu") (net 84))
   (segment (start 96.5215 88.6975) (end 97.636 89.812) (width 0.254) (layer "F.Cu") (net 84))
-  (segment (start 83.82 46) (end 83.82 44.45) (width 0.254) (layer "F.Cu") (net 95))
-  (via (at 83.82 44.45) (size 0.8) (drill 0.4) (layers "F.Cu" "B.Cu") (net 95))
-  (segment (start 83.82 44.45) (end 86.052 42.218) (width 0.254) (layer "B.Cu") (net 95))
-  (segment (start 86.052 42.218) (end 92.456 42.218) (width 0.254) (layer "B.Cu") (net 95))
-  (segment (start 87.63 46) (end 87.63 44.45) (width 0.254) (layer "F.Cu") (net 96))
-  (via (at 87.63 44.45) (size 0.8) (drill 0.4) (layers "F.Cu" "B.Cu") (net 96))
-  (segment (start 88.392 43.688) (end 87.63 44.45) (width 0.254) (layer "B.Cu") (net 96))
-  (segment (start 88.392 43.688) (end 92.456 43.688) (width 0.254) (layer "B.Cu") (net 96))
-  (segment (start 88.9 46) (end 88.9 44.45) (width 0.254) (layer "F.Cu") (net 98))
-  (via (at 88.9 44.45) (size 0.8) (drill 0.4) (layers "F.Cu" "B.Cu") (net 98))
-  (segment (start 88.9 44.45) (end 92.456 44.45) (width 0.254) (layer "B.Cu") (net 98))
-  (segment (start 77.47 46) (end 77.47 44.45) (width 0.254) (layer "F.Cu") (net 104))
-  (via (at 77.47 44.45) (size 0.8) (drill 0.4) (layers "F.Cu" "B.Cu") (net 104))
-  (segment (start 82.296 39.624) (end 92.456 39.624) (width 0.254) (layer "B.Cu") (net 104))
-  (segment (start 77.47 44.45) (end 82.296 39.624) (width 0.254) (layer "B.Cu") (net 104))
-  (segment (start 78.74 46) (end 78.74 44.45) (width 0.254) (layer "F.Cu") (net 105))
-  (via (at 78.74 44.45) (size 0.8) (drill 0.4) (layers "F.Cu" "B.Cu") (net 105))
-  (segment (start 83.058 40.132) (end 92.456 40.132) (width 0.254) (layer "B.Cu") (net 105))
-  (segment (start 78.74 44.45) (end 83.058 40.132) (width 0.254) (layer "B.Cu") (net 105))
 )
