File: boardlock/_autosave-power.kicad_sch (KiCad schematic)
At the start: 26 parts, among them U6 TPS630701RNMR, U7 MCP1661

Commit message: buck-boost WIP
Connections:
- net VAUX: now reaches C18.1, U6.3 (VAUX)
Changed lines of the file:
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@@
     (effects (font (size 1.27 1.27)) (justify left bottom))
+  )
+  (label "VAUX" (at 144.78 104.14 180) (fields_autoplaced)
+    (effects (font (size 1.27 1.27)) (justify right bottom))
   )
   (label "Buck_Boost_FB" (at 200.66 81.28 180) (fields_autoplaced)
     (effects (font (size 1.27 1.27)) (justify right bottom))
   )
-  (label "VSEL" (at 144.78 99.06 180) (fields_autoplaced)
-    (effects (font (size 1.27 1.27)) (justify right bottom))
-  )
